File: Hardware/tool_circuit/Pi_Connection.sch (KiCad schematic (older format))
At the start: 0 parts

Commit message: Pi hat
Changed lines of the file:
@@
 $Descr A4 11693 8268
 encoding utf-8
-Sheet 4 5
+Sheet 4 6
 Title ""
 Date ""
@@
 Comment4 ""
 $EndDescr
-Text HLabel 9400 2400 0    50   BiDi ~ 0
+Text HLabel 2000 2200 0    50   BiDi ~ 0
 DATA
+$Sheet
+S 2600 1850 1300 1000
+U 612AC45A
+F0 "Pi_Hat" 50
+F1 "Pi_Hat.sch" 50
+$EndSheet
+Wire Bus Line
+	2000 2200 2700 2200
 $EndSCHEMATC

Commit message: regulator/other changes
Changed lines of the file:
@@
 $Descr A4 11693 8268
 encoding utf-8
-Sheet 4 6
+Sheet 4 7
 Title ""
 Date ""
@@
 Comment4 ""
 $EndDescr
-Text HLabel 2000 2200 0    50   BiDi ~ 0
+Text HLabel 2600 2250 2    50   BiDi ~ 0
 DATA
 $Sheet
@@
 F1 "Pi_Hat.sch" 50
 $EndSheet
-Wire Bus Line
-	2000 2200 2700 2200
+Text HLabel 2600 2450 2    50   Input ~ 0
+5V
 $EndSCHEMATC
