File: Hardware/tool_circuit/Temp_Sense.sch (KiCad schematic (older format))
At the start: 1 part

Commit message: temp sensor
Parts:
- added R?: 5K, symbol Device:R
Connections:
- net labels added: GND
- wire segments 2 -> 5
Other:
- moved on the sheet: U?
Changed lines of the file:
@@
 	6350 3850 6250 3750
 Wire Wire Line
-	6250 3750 5400 3750
-Wire Bus Line
-	6350 3550 6350 4250
+	6250 3750 5800 3750
 Wire Wire Line
-	3400 2950 3400 3250
+	5100 3150 5100 3450
 $Comp
 L power:+3.3V #PWR?
 U 1 1 611F0935
-P 3400 2950
-F 0 "#PWR?" H 3400 2800 50  0001 C CNN
-F 1 "+3.3V" H 3415 3123 50  0000 C CNN
-F 2 "" H 3400 2950 50  0001 C CNN
-F 3 "" H 3400 2950 50  0001 C CNN
-	1    3400 2950
+P 5100 3150
+F 0 "#PWR?" H 5100 3000 50  0001 C CNN
+F 1 "+3.3V" H 5115 3323 50  0000 C CNN
+F 2 "" H 5100 3150 50  0001 C CNN
+F 3 "" H 5100 3150 50  0001 C CNN
+	1    5100 3150
 	1    0    0    -1
 $EndComp
@@
 L Sensor:DHT11 U?
 U 1 1 611EBA26
-P 3400 3550
+P 5100 3750
 AR Path="/611EBA26" Ref="U?"  Part="1"
 AR Path="/611DBC89/611EBA26" Ref="U?"  Part="1"
-F 0 "U?" H 3156 3596 50  0000 R CNN
-F 1 "DHT11" H 3156 3505 50  0000 R CNN
-F 2 "Sensor:Aosong_DHT11_5.5x12.0_P2.54mm" H 3400 3150 50  0001 C CNN
-F 3 "http://akizukidenshi.com/download/ds/aosong/DHT11.pdf" H 3550 3800 50  0001 C CNN
-	1    3400 3550
+F 0 "U?" H 4856 3796 50  0000 R CNN
+F 1 "DHT11" H 4856 3705 50  0000 R CNN
+F 2 "Sensor:Aosong_DHT11_5.5x12.0_P2.54mm" H 5100 3350 50  0001 C CNN
+F 3 "http://akizukidenshi.com/download/ds/aosong/DHT11.pdf" H 5250 4000 50  0001 C CNN
+	1    5100 3750
 	1    0    0    -1
 $EndComp
+$Comp
+L power:+3.3V #PWR?
+U 1 1 6122E57C
+P 5800 3150
+F 0 "#PWR?" H 5800 3000 50  0001 C CNN
+F 1 "+3.3V" H 5815 3323 50  0000 C CNN
+F 2 "" H 5800 3150 50  0001 C CNN
+F 3 "" H 5800 3150 50  0001 C CNN
+	1    5800 3150
+	1    0    0    -1
+$EndComp
+Wire Wire Line
+	5800 3150 5800 3250
+Connection ~ 5800 3750
+Wire Wire Line
+	5800 3750 5400 3750
+$Comp
+L Device:R R?
+U 1 1 612305FD
+P 5800 3400
+F 0 "R?" H 5870 3446 50  0000 L CNN
+F 1 "5K" H 5870 3355 50  0000 L CNN
+F 2 "" V 5730 3400 50  0001 C CNN
+F 3 "~" H 5800 3400 50  0001 C CNN
+	1    5800 3400
+	1    0    0    -1
+$EndComp
+Wire Wire Line
+	5800 3550 5800 3750
+Wire Bus Line
+	6350 3550 6350 4250
+$Comp
+L power:GND #PWR?
+U 1 1 61232568
+P 5100 4050
+F 0 "#PWR?" H 5100 3800 50  0001 C CNN
+F 1 "GND" H 5105 3877 50  0000 C CNN
+F 2 "" H 5100 4050 50  0001 C CNN
+F 3 "" H 5100 4050 50  0001 C CNN
+	1    5100 4050
+	1    0    0    -1
+$EndComp

Commit message: symbols
Parts:
- removed R?: 5K, symbol Device:R
- added R1: RNCP1206FTD4K99, STA_RNCP1206_STP, symbol 2021-09-15_14-25-04:RNCP1206FTD4K99
- gave numbers to parts that had none: 1
Changed lines of the file:
@@
 $Descr A4 11693 8268
 encoding utf-8
-Sheet 2 7
+Sheet 2 5
 Title ""
 Date ""
@@
 	5100 3150 5100 3450
 $Comp
-L power:+3.3V #PWR?
+L power:+3.3V #PWR0102
 U 1 1 611F0935
 P 5100 3150
-F 0 "#PWR?" H 5100 3000 50  0001 C CNN
+F 0 "#PWR0102" H 5100 3000 50  0001 C CNN
 F 1 "+3.3V" H 5115 3323 50  0000 C CNN
 F 2 "" H 5100 3150 50  0001 C CNN
@@
 P 5100 3750
 AR Path="/611EBA26" Ref="U?"  Part="1"
-AR Path="/611DBC89/611EBA26" Ref="U?"  Part="1"
-F 0 "U?" H 4856 3796 50  0000 R CNN
+AR Path="/611DBC89/611EBA26" Ref="U1"  Part="1"
+F 0 "U1" H 4856 3796 50  0000 R CNN
 F 1 "DHT11" H 4856 3705 50  0000 R CNN
 F 2 "Sensor:Aosong_DHT11_5.5x12.0_P2.54mm" H 5100 3350 50  0001 C CNN
@@
 $EndComp
 $Comp
-L power:+3.3V #PWR?
+L power:+3.3V #PWR0103
 U 1 1 6122E57C
-P 5800 3150
-F 0 "#PWR?" H 5800 3000 50  0001 C CNN
-F 1 "+3.3V" H 5815 3323 50  0000 C CNN
-F 2 "" H 5800 3150 50  0001 C CNN
-F 3 "" H 5800 3150 50  0001 C CNN
-	1    5800 3150
+P 5800 3050
+F 0 "#PWR0103" H 5800 2900 50  0001 C CNN
+F 1 "+3.3V" H 5800 3200 50  0000 C CNN
+F 2 "" H 5800 3050 50  0001 C CNN
+F 3 "" H 5800 3050 50  0001 C CNN
+	1    5800 3050
 	1    0    0    -1
 $EndComp
@@
 Wire Wire Line
 	5800 3750 5400 3750
-$Comp
-L Device:R R?
-U 1 1 612305FD
-P 5800 3400
-F 0 "R?" H 5870 3446 50  0000 L CNN
-F 1 "5K" H 5870 3355 50  0000 L CNN
-F 2 "" V 5730 3400 50  0001 C CNN
-F 3 "~" H 5800 3400 50  0001 C CNN
-	1    5800 3400
-	1    0    0    -1
-$EndComp
 Wire Wire Line
 	5800 3550 5800 3750
 $Comp
-L power:GND #PWR?
+L power:GND #PWR0104
 U 1 1 61232568
 P 5100 4050
-F 0 "#PWR?" H 5100 3800 50  0001 C CNN
+F 0 "#PWR0104" H 5100 3800 50  0001 C CNN
 F 1 "GND" H 5105 3877 50  0000 C CNN
 F 2 "" H 5100 4050 50  0001 C CNN
@@
 	1    0    0    -1
 $EndComp
+$Comp
+L 2021-09-15_14-25-04:RNCP1206FTD4K99 R1
+U 1 1 614256D6
+P 5800 3050
+F 0 "R1" H 6050 3288 60  0000 C CNN
+F 1 "RNCP1206FTD4K99" H 6050 3182 60  0000 C CNN
+F 2 "STA_RNCP1206_STP" H 6050 2715 60  0001 C CNN
+F 3 "" H 5800 3050 60  0000 C CNN
+	1    5800 3050
+	0    1    1    0
+$EndComp
 Wire Bus Line

Commit message: symbolsssss
Parts:
- R1: symbol 2021-09-15_14-25-04:RNCP1206FTD4K99 -> tool_circuit-rescue:RNCP1206FTD4K99-2021-09-15_14-25-04
Changed lines of the file:
@@
 $EndComp
 $Comp
-L 2021-09-15_14-25-04:RNCP1206FTD4K99 R1
+L tool_circuit-rescue:RNCP1206FTD4K99-2021-09-15_14-25-04 R1
 U 1 1 614256D6
 P 5800 3050
+AR Path="/614256D6" Ref="R1"  Part="1"
+AR Path="/611DBC89/614256D6" Ref="R1"  Part="1"
 F 0 "R1" H 6050 3288 60  0000 C CNN
 F 1 "RNCP1206FTD4K99" H 6050 3182 60  0000 C CNN

Commit message: updated symbols/footprint paths for today
Parts:
- R1: footprint STA_RNCP1206_STP -> RNCP1206FTD4K99:RNCP1206FTD4K99
Changed lines of the file:
@@
 $Descr A4 11693 8268
 encoding utf-8
-Sheet 2 5
+Sheet 5 5
 Title ""
 Date ""
@@
 F 0 "R1" H 6050 3288 60  0000 C CNN
 F 1 "RNCP1206FTD4K99" H 6050 3182 60  0000 C CNN
-F 2 "STA_RNCP1206_STP" H 6050 2715 60  0001 C CNN
+F 2 "RNCP1206FTD4K99:RNCP1206FTD4K99" H 6050 2715 60  0001 C CNN
 F 3 "" H 5800 3050 60  0000 C CNN
 	1    5800 3050
