File: Hardware/tool_circuit/Temp_Sense.sch (KiCad schematic (older format))
At the start: 2 parts, among them U1 DHT11

Commit message: pcb layout and schematic changes
Parts:
- removed R1: RNCP1206FTD4K99, RNCP1206FTD4K99:RNCP1206FTD4K99, symbol tool_circuit-rescue:RNCP1206FTD4K99-2021-09-15_14-25-04
- removed U1: DHT11, Sensor:Aosong_DHT11_5.5x12.0_P2.54mm, symbol Sensor:DHT11
- added J3: Conn_01x03_Female, Connector_PinHeader_2.54mm:PinHeader_1x03_P2.54mm_Vertical, symbol Connector:Conn_01x03_Female
Connections:
- net labels added: +5V, GPIO_17
- net labels removed: +3.3V, TEMP_DATA
- wire segments 5 -> 3
Changed lines of the file:
@@
 $Descr A4 11693 8268
 encoding utf-8
-Sheet 5 6
+Sheet 5 7
 Title ""
 Date ""
@@
 Comment4 ""
 $EndDescr
-Text HLabel 6800 3550 2    50   BiDi ~ 0
-TEMP_DATA
-Wire Bus Line
-	6800 3550 6350 3550
-Entry Wire Line
-	6350 3850 6250 3750
-Wire Wire Line
-	6250 3750 5800 3750
-Wire Wire Line
-	5100 3150 5100 3450
 $Comp
-L power:+3.3V #PWR0102
-U 1 1 611F0935
-P 5100 3150
-F 0 "#PWR0102" H 5100 3000 50  0001 C CNN
-F 1 "+3.3V" H 5115 3323 50  0000 C CNN
-F 2 "" H 5100 3150 50  0001 C CNN
-F 3 "" H 5100 3150 50  0001 C CNN
-	1    5100 3150
+L Connector:Conn_01x03_Female J3
+U 1 1 614AEC17
+P 5700 3500
+F 0 "J3" H 5728 3526 50  0000 L CNN
+F 1 "Conn_01x03_Female" H 5728 3435 50  0000 L CNN
+F 2 "Connector_PinHeader_2.54mm:PinHeader_1x03_P2.54mm_Vertical" H 5700 3500 50  0001 C CNN
+F 3 "~" H 5700 3500 50  0001 C CNN
+	1    5700 3500
 	1    0    0    -1
 $EndComp
 $Comp
-L Sensor:DHT11 U?
-U 1 1 611EBA26
-P 5100 3750
-AR Path="/611EBA26" Ref="U?"  Part="1"
-AR Path="/611DBC89/611EBA26" Ref="U1"  Part="1"
-F 0 "U1" H 4856 3796 50  0000 R CNN
-F 1 "DHT11" H 4856 3705 50  0000 R CNN
-F 2 "Sensor:Aosong_DHT11_5.5x12.0_P2.54mm" H 5100 3350 50  0001 C CNN
-F 3 "http://akizukidenshi.com/download/ds/aosong/DHT11.pdf" H 5250 4000 50  0001 C CNN
-	1    5100 3750
-	1    0    0    -1
-$EndComp
-$Comp
-L power:+3.3V #PWR0103
-U 1 1 6122E57C
-P 5800 3050
-F 0 "#PWR0103" H 5800 2900 50  0001 C CNN
-F 1 "+3.3V" H 5800 3200 50  0000 C CNN
-F 2 "" H 5800 3050 50  0001 C CNN
-F 3 "" H 5800 3050 50  0001 C CNN
-	1    5800 3050
+L power:GND #PWR0102
+U 1 1 614AF32D
+P 5350 3700
+F 0 "#PWR0102" H 5350 3450 50  0001 C CNN
+F 1 "GND" H 5355 3527 50  0000 C CNN
+F 2 "" H 5350 3700 50  0001 C CNN
+F 3 "" H 5350 3700 50  0001 C CNN
+	1    5350 3700
 	1    0    0    -1
 $EndComp
 Wire Wire Line
-	5800 3150 5800 3250
-Connection ~ 5800 3750
+	5500 3600 5350 3600
 Wire Wire Line
-	5800 3750 5400 3750
-Wire Wire Line
-	5800 3550 5800 3750
+	5350 3600 5350 3700
 $Comp
-L power:GND #PWR0104
-U 1 1 61232568
-P 5100 4050
-F 0 "#PWR0104" H 5100 3800 50  0001 C CNN
-F 1 "GND" H 5105 3877 50  0000 C CNN
-F 2 "" H 5100 4050 50  0001 C CNN
-F 3 "" H 5100 4050 50  0001 C CNN
-	1    5100 4050
+L power:+5V #PWR0103
+U 1 1 614AFBC4
+P 5050 3400
+F 0 "#PWR0103" H 5050 3250 50  0001 C CNN
+F 1 "+5V" H 5065 3573 50  0000 C CNN
+F 2 "" H 5050 3400 50  0001 C CNN
+F 3 "" H 5050 3400 50  0001 C CNN
+	1    5050 3400
 	1    0    0    -1
 $EndComp
-$Comp
-L tool_circuit-rescue:RNCP1206FTD4K99-2021-09-15_14-25-04 R1
-U 1 1 614256D6
-P 5800 3050
-AR Path="/614256D6" Ref="R1"  Part="1"
-AR Path="/611DBC89/614256D6" Ref="R1"  Part="1"
-F 0 "R1" H 6050 3288 60  0000 C CNN
-F 1 "RNCP1206FTD4K99" H 6050 3182 60  0000 C CNN
-F 2 "RNCP1206FTD4K99:RNCP1206FTD4K99" H 6050 2715 60  0001 C CNN
-F 3 "" H 5800 3050 60  0000 C CNN
-	1    5800 3050
-	0    1    1    0
-$EndComp
-Wire Bus Line
-	6350 3550 6350 4250
+Wire Wire Line
+	5050 3400 5500 3400
+Text HLabel 5500 3500 0    50   BiDi ~ 0
+GPIO_17
 $EndSCHEMATC
