File: Hardware/tool_circuit/Vibration_Sensor.sch (KiCad schematic (older format))
At the start: 0 parts

Commit message: updated symbols/footprint paths for today
Changed lines of the file:
@@
 Comment4 ""
 $EndDescr
-Text HLabel 5400 2600 0    50   BiDi ~ 0
+Text HLabel 4900 3100 0    50   BiDi ~ 0
 VIB_DATA
 $EndSCHEMATC

Commit message: edited proposal doc + started pcb layout
Parts:
- added J1: Conn_01x03_Female, Connector_PinHeader_2.54mm:PinHeader_1x03_P2.54mm_Vertical, symbol Connector:Conn_01x03_Female
Changed lines of the file:
@@
 $Descr A4 11693 8268
 encoding utf-8
-Sheet 3 5
+Sheet 2 6
 Title ""
 Date ""
@@
 Comment4 ""
 $EndDescr
-Text HLabel 4900 3100 0    50   BiDi ~ 0
+Text HLabel 4250 2950 0    50   BiDi ~ 0
 VIB_DATA
+$Comp
+L Connector:Conn_01x03_Female J1
+U 1 1 6144B415
+P 5000 3100
+F 0 "J1" H 5028 3126 50  0000 L CNN
+F 1 "Conn_01x03_Female" H 5028 3035 50  0000 L CNN
+F 2 "Connector_PinHeader_2.54mm:PinHeader_1x03_P2.54mm_Vertical" H 5000 3100 50  0001 C CNN
+F 3 "~" H 5000 3100 50  0001 C CNN
+	1    5000 3100
+	1    0    0    -1
+$EndComp
 $EndSCHEMATC

Commit message: pcb layout and schematic changes
Connections:
- net +5V: now reaches J1.1 (Pin_1)
- net GPIO_27: now reaches J1.2 (Pin_2)
- net GND: now reaches J1.3 (Pin_3)
Other:
- moved on the sheet: J1
Changed lines of the file:
@@
 $Descr A4 11693 8268
 encoding utf-8
-Sheet 2 6
+Sheet 2 7
 Title ""
 Date ""
@@
 Comment4 ""
 $EndDescr
-Text HLabel 4250 2950 0    50   BiDi ~ 0
-VIB_DATA
+Text HLabel 5350 3100 0    50   BiDi ~ 0
+GPIO_27
 $Comp
 L Connector:Conn_01x03_Female J1
 U 1 1 6144B415
-P 5000 3100
-F 0 "J1" H 5028 3126 50  0000 L CNN
-F 1 "Conn_01x03_Female" H 5028 3035 50  0000 L CNN
-F 2 "Connector_PinHeader_2.54mm:PinHeader_1x03_P2.54mm_Vertical" H 5000 3100 50  0001 C CNN
-F 3 "~" H 5000 3100 50  0001 C CNN
-	1    5000 3100
+P 5550 3100
+F 0 "J1" H 5578 3126 50  0000 L CNN
+F 1 "Conn_01x03_Female" H 5578 3035 50  0000 L CNN
+F 2 "Connector_PinHeader_2.54mm:PinHeader_1x03_P2.54mm_Vertical" H 5550 3100 50  0001 C CNN
+F 3 "~" H 5550 3100 50  0001 C CNN
+	1    5550 3100
 	1    0    0    -1
 $EndComp
+$Comp
+L power:GND #PWR0105
+U 1 1 614A4174
+P 5150 3200
+F 0 "#PWR0105" H 5150 2950 50  0001 C CNN
+F 1 "GND" H 5155 3027 50  0000 C CNN
+F 2 "" H 5150 3200 50  0001 C CNN
+F 3 "" H 5150 3200 50  0001 C CNN
+	1    5150 3200
+	1    0    0    -1
+$EndComp
+Wire Wire Line
+	5350 3200 5150 3200
+Wire Wire Line
+	5100 2950 5100 3000
+Wire Wire Line
+	5100 3000 5350 3000
+$Comp
+L power:+5V #PWR0106
+U 1 1 614A5231
+P 5100 2950
+F 0 "#PWR0106" H 5100 2800 50  0001 C CNN
+F 1 "+5V" H 5115 3123 50  0000 C CNN
+F 2 "" H 5100 2950 50  0001 C CNN
+F 3 "" H 5100 2950 50  0001 C CNN
+	1    5100 2950
+	1    0    0    -1
+$EndComp
