File: Hardware/tool_circuit/Accelerometer copy.sch (KiCad schematic (older format))
At the start: 1 part

Commit message: schematic revisions
Parts:
- gave numbers to parts that had none: 1
Changed lines of the file:
@@
 $Descr A4 11693 8268
 encoding utf-8
-Sheet 7 8
+Sheet 6 8
 Title ""
 Date ""
@@
 	5450 4300 5550 4200
 $Comp
-L Connector:Conn_01x08_Female J?
+L Connector:Conn_01x08_Female J1
 U 1 1 6149E3EA
 P 6200 3600
-F 0 "J?" H 6228 3576 50  0000 L CNN
+F 0 "J1" H 6228 3576 50  0000 L CNN
 F 1 "Conn_01x08_Female" H 6228 3485 50  0000 L CNN
 F 2 "Connector_PinHeader_2.54mm:PinHeader_1x08_P2.54mm_Vertical" H 6200 3600 50  0001 C CNN
@@
 	5100 3300 6000 3300
 $Comp
-L power:+3.3V #PWR?
+L power:+3.3V #PWR07
 U 1 1 614A0E05
 P 5300 3750
-F 0 "#PWR?" H 5300 3600 50  0001 C CNN
+F 0 "#PWR07" H 5300 3600 50  0001 C CNN
 F 1 "+3.3V" H 5315 3923 50  0000 C CNN
 F 2 "" H 5300 3750 50  0001 C CNN
@@
 $EndComp
 $Comp
-L power:GND #PWR?
+L power:GND #PWR06
 U 1 1 6149F537
 P 5100 3750
-F 0 "#PWR?" H 5100 3500 50  0001 C CNN
+F 0 "#PWR06" H 5100 3500 50  0001 C CNN
 F 1 "GND" H 5105 3577 50  0000 C CNN
 F 2 "" H 5100 3750 50  0001 C CNN
