File: Hardware/tool_circuit/Time_of_Use.sch (KiCad schematic (older format))
At the start: 1 part, among them J1 Conn_01x03_Female

Commit message: Tool Circuit schematic updates
Parts:
- removed J1: Conn_01x03_Female, Connector_PinHeader_2.54mm:PinHeader_1x03_P2.54mm_Vertical, symbol Connector:Conn_01x03_Female
- added R4: RMCF1206JT150R, RESC3216X70N, symbol RMCF1206JT150R:RMCF1206JT150R
- added U2: ADG419BN, Package_DIP:DIP-8_W7.62mm, symbol Analog_Switch:ADG419BN
Connections:
- net labels added: GPIO17, GPIO[17..17]
- net labels removed: GPIO_27
- wire segments 3 -> 5
Changed lines of the file:
@@
 $Descr A4 11693 8268
 encoding utf-8
-Sheet 2 7
+Sheet 7 8
 Title ""
 Date ""
@@
 Comment4 ""
 $EndDescr
-Text HLabel 4650 3450 0    50   BiDi ~ 0
-GPIO_27
-Wire Wire Line
-	4400 3300 4400 3350
-Wire Wire Line
-	4400 3350 4650 3350
 $Comp
-L power:+5V #PWR0106
+L power:+5V #PWR09
 U 1 1 614A5231
-P 4400 3300
-F 0 "#PWR0106" H 4400 3150 50  0001 C CNN
-F 1 "+5V" H 4415 3473 50  0000 C CNN
-F 2 "" H 4400 3300 50  0001 C CNN
-F 3 "" H 4400 3300 50  0001 C CNN
-	1    4400 3300
+P 6350 3550
+F 0 "#PWR09" H 6350 3400 50  0001 C CNN
+F 1 "+5V" H 6365 3723 50  0000 C CNN
+F 2 "" H 6350 3550 50  0001 C CNN
+F 3 "" H 6350 3550 50  0001 C CNN
+	1    6350 3550
+	1    0    0    -1
+$EndComp
+$Comp
+L power:GND #PWR08
+U 1 1 614A4174
+P 4950 5050
+F 0 "#PWR08" H 4950 4800 50  0001 C CNN
+F 1 "GND" H 4955 4877 50  0000 C CNN
+F 2 "" H 4950 5050 50  0001 C CNN
+F 3 "" H 4950 5050 50  0001 C CNN
+	1    4950 5050
+	1    0    0    -1
+$EndComp
+$Comp
+L RMCF1206JT150R:RMCF1206JT150R R4
+U 1 1 614C1CF4
+P 4950 4650
+F 0 "R4" V 4904 4755 50  0000 L CNN
+F 1 "RMCF1206JT150R" V 4995 4755 50  0000 L CNN
+F 2 "RESC3216X70N" H 4950 4650 50  0001 L BNN
+F 3 "" H 4950 4650 50  0001 L BNN
+	1    4950 4650
+	0    1    1    0
+$EndComp
+$Comp
+L Analog_Switch:ADG419BN U2
+U 1 1 614CBD1C
+P 5550 4050
+F 0 "U2" H 5550 4292 50  0000 C CNN
+F 1 "ADG419BN" H 5550 4201 50  0000 C CNN
+F 2 "Package_DIP:DIP-8_W7.62mm" H 5550 3750 50  0001 C CNN
+F 3 "https://www.analog.com/media/en/technical-documentation/data-sheets/ADG419.pdf" H 5550 3850 50  0001 C CNN
+	1    5550 4050
 	1    0    0    -1
 $EndComp
 Wire Wire Line
-	4650 3550 4450 3550
-$Comp
-L Connector:Conn_01x03_Female J1
-U 1 1 6144B415
-P 4850 3450
-F 0 "J1" H 4878 3476 50  0000 L CNN
-F 1 "Conn_01x03_Female" H 4878 3385 50  0000 L CNN
-F 2 "Connector_PinHeader_2.54mm:PinHeader_1x03_P2.54mm_Vertical" H 4850 3450 50  0001 C CNN
-F 3 "~" H 4850 3450 50  0001 C CNN
-	1    4850 3450
-	1    0    0    -1
-$EndComp
-$Comp
-L power:GND #PWR0105
-U 1 1 614A4174
-P 4450 3550
-F 0 "#PWR0105" H 4450 3300 50  0001 C CNN
-F 1 "GND" H 4455 3377 50  0000 C CNN
-F 2 "" H 4450 3550 50  0001 C CNN
-F 3 "" H 4450 3550 50  0001 C CNN
-	1    4450 3550
-	1    0    0    -1
-$EndComp
+	4950 4150 4950 4250
+Wire Wire Line
+	4950 4150 5250 4150
+Connection ~ 4950 4150
+Wire Wire Line
+	6350 4050 5850 4050
+Wire Wire Line
+	6350 3550 6350 4050
+Wire Wire Line
+	3950 4150 4950 4150
+Text Label 4150 4150 0    50   ~ 0
+GPIO17
+Entry Wire Line
+	3850 4050 3950 4150
+Text Label 3650 3900 0    50   ~ 0
+GPIO[17..17]
+Wire Bus Line
+	3850 3900 3850 4350
+Wire Bus Line
+	3650 3900 3850 3900
+Text HLabel 3650 3900 0    50   Input ~ 0
+GPIO17
 $EndSCHEMATC

Commit message: schematic LEDs + switch
Parts:
- removed U2: ADG419BN, Package_DIP:DIP-8_W7.62mm, symbol Analog_Switch:ADG419BN
- added LED1: 151034BS03000, LED_BS03000_WRE, symbol 2021-09-28_17-07-40:151034BS03000
- added R7: RC1206JR-07110RL, RESC3116X65N, symbol RC1206JR-07110RL:RC1206JR-07110RL
- added S1: 1825255-1, SW_1825255-1, symbol 1825255-1:1825255-1
Connections:
- net labels added: GPIO17_22, GPIO22, GPIO[17..22]
- net labels removed: GPIO[17..17]
- wire segments 5 -> 14
Changed lines of the file:
@@
 L power:+5V #PWR07
 U 1 1 614A5231
-P 6350 3550
-F 0 "#PWR07" H 6350 3400 50  0001 C CNN
-F 1 "+5V" H 6365 3723 50  0000 C CNN
-F 2 "" H 6350 3550 50  0001 C CNN
-F 3 "" H 6350 3550 50  0001 C CNN
-	1    6350 3550
+P 6650 3500
+F 0 "#PWR07" H 6650 3350 50  0001 C CNN
+F 1 "+5V" H 6665 3673 50  0000 C CNN
+F 2 "" H 6650 3500 50  0001 C CNN
+F 3 "" H 6650 3500 50  0001 C CNN
+	1    6650 3500
 	1    0    0    -1
 $EndComp
@@
 	0    1    1    0
 $EndComp
-$Comp
-L Analog_Switch:ADG419BN U2
-U 1 1 614CBD1C
-P 5550 4050
-F 0 "U2" H 5550 4292 50  0000 C CNN
-F 1 "ADG419BN" H 5550 4201 50  0000 C CNN
-F 2 "Package_DIP:DIP-8_W7.62mm" H 5550 3750 50  0001 C CNN
-F 3 "https://www.analog.com/media/en/technical-documentation/data-sheets/ADG419.pdf" H 5550 3850 50  0001 C CNN
-	1    5550 4050
-	1    0    0    -1
-$EndComp
 Wire Wire Line
 	4950 4150 4950 4250
-Wire Wire Line
-	4950 4150 5250 4150
 Connection ~ 4950 4150
 Wire Wire Line
-	6350 4050 5850 4050
+	6650 4000 6150 4000
 Wire Wire Line
-	6350 3550 6350 4050
+	6650 3500 6650 3650
 Wire Wire Line
 	3950 4150 4950 4150
@@
 	3850 4050 3950 4150
 Text Label 3650 3900 0    50   ~ 0
-GPIO[17..17]
+GPIO[17..22]
 Wire Bus Line
 	3650 3900 3850 3900
 Text HLabel 3650 3900 0    50   Input ~ 0
-GPIO17
+GPIO17_22
+$Comp
+L 2021-09-28_17-07-40:151034BS03000 LED1
+U 1 1 615638DB
+P 7200 4000
+F 0 "LED1" V 7347 4228 60  0000 L CNN
+F 1 "151034BS03000" V 7453 4228 60  0000 L CNN
+F 2 "LED_BS03000_WRE" H 7400 3640 60  0001 C CNN
+F 3 "" H 7200 4000 60  0000 C CNN
+	1    7200 4000
+	0    1    1    0
+$EndComp
+Wire Wire Line
+	6650 3650 7200 3650
+Wire Wire Line
+	7200 3650 7200 4000
+Connection ~ 6650 3650
+Wire Wire Line
+	6650 3650 6650 4000
+$Comp
+L RC1206JR-07110RL:RC1206JR-07110RL R7
+U 1 1 6156637C
+P 7200 4800
+F 0 "R7" V 7154 4905 50  0000 L CNN
+F 1 "RC1206JR-07110RL" V 7245 4905 50  0000 L CNN
+F 2 "RESC3116X65N" H 7200 4800 50  0001 L BNN
+F 3 "" H 7200 4800 50  0001 L BNN
+	1    7200 4800
+	0    1    1    0
+$EndComp
+Entry Wire Line
+	3850 4200 3950 4300
+Wire Wire Line
+	3950 4300 3950 5450
+Wire Wire Line
+	3950 5450 7200 5450
+Text Label 3950 4550 0    50   ~ 0
+GPIO22
+$Comp
+L 1825255-1:1825255-1 S1
+U 1 1 61568B03
+P 5800 4250
+F 0 "S1" H 6030 4296 50  0000 L CNN
+F 1 "1825255-1" H 6030 4205 50  0000 L CNN
+F 2 "SW_1825255-1" H 5800 4250 50  0001 L BNN
+F 3 "" H 5800 4250 50  0001 L BNN
+F 4 "1825255-1" H 5800 4250 50  0001 L BNN "Comment"
+	1    5800 4250
+	1    0    0    -1
+$EndComp
+Wire Wire Line
+	7200 5450 7200 5200
+Wire Wire Line
+	4950 4150 5400 4150
+Wire Wire Line
+	6150 4000 6150 3850
+Wire Wire Line
+	6150 3850 5400 3850
+Wire Wire Line
+	5400 3850 5400 4050
 Wire Bus Line
 	3850 3900 3850 4350

Commit message: made some post review changes
Connections:
- net labels added: TIME_OF_USE_DATA
- net labels removed: GPIO17_22, GPIO[17..22]
- no-connect marks 0 -> 1
Changed lines of the file:
@@
 Entry Wire Line
 	3850 4050 3950 4150
-Text Label 3650 3900 0    50   ~ 0
-GPIO[17..22]
 Wire Bus Line
 	3650 3900 3850 3900
-Text HLabel 3650 3900 0    50   Input ~ 0
-GPIO17_22
 $Comp
 L 2021-09-28_17-07-40:151034BS03000 LED1
@@
 Wire Wire Line
 	5400 3850 5400 4050
+NoConn ~ 5400 4250
 Wire Bus Line
 	3850 3900 3850 4350
+Text HLabel 3650 3900 0    50   BiDi ~ 0
+TIME_OF_USE_DATA
 $EndSCHEMATC

Commit message: Latest revisions to schematic
Parts:
- removed LED1: 151034BS03000, LED_BS03000_WRE, symbol 2021-09-28_17-07-40:151034BS03000
- removed R4: RMCF1206JT150R, RESC3216X70N, symbol RMCF1206JT150R:RMCF1206JT150R
- removed R7: RC1206JR-07110RL, RESC3116X65N, symbol RC1206JR-07110RL:RC1206JR-07110RL
Connections:
- net labels removed: GND, GPIO22
- wire segments 14 -> 6
Changed lines of the file:
@@
 	1    0    0    -1
 $EndComp
-$Comp
-L power:GND #PWR06
-U 1 1 614A4174
-P 4950 5050
-F 0 "#PWR06" H 4950 4800 50  0001 C CNN
-F 1 "GND" H 4955 4877 50  0000 C CNN
-F 2 "" H 4950 5050 50  0001 C CNN
-F 3 "" H 4950 5050 50  0001 C CNN
-	1    4950 5050
-	1    0    0    -1
-$EndComp
-$Comp
-L RMCF1206JT150R:RMCF1206JT150R R4
-U 1 1 614C1CF4
-P 4950 4650
-F 0 "R4" V 4904 4755 50  0000 L CNN
-F 1 "RMCF1206JT150R" V 4995 4755 50  0000 L CNN
-F 2 "RESC3216X70N" H 4950 4650 50  0001 L BNN
-F 3 "" H 4950 4650 50  0001 L BNN
-	1    4950 4650
-	0    1    1    0
-$EndComp
-Wire Wire Line
-	4950 4150 4950 4250
-Connection ~ 4950 4150
 Wire Wire Line
 	6650 4000 6150 4000
-Wire Wire Line
-	6650 3500 6650 3650
-Wire Wire Line
-	3950 4150 4950 4150
 Text Label 4150 4150 0    50   ~ 0
 GPIO17
@@
 Wire Bus Line
 	3650 3900 3850 3900
-$Comp
-L 2021-09-28_17-07-40:151034BS03000 LED1
-U 1 1 615638DB
-P 7200 4000
-F 0 "LED1" V 7347 4228 60  0000 L CNN
-F 1 "151034BS03000" V 7453 4228 60  0000 L CNN
-F 2 "LED_BS03000_WRE" H 7400 3640 60  0001 C CNN
-F 3 "" H 7200 4000 60  0000 C CNN
-	1    7200 4000
-	0    1    1    0
-$EndComp
-Wire Wire Line
-	6650 3650 7200 3650
-Wire Wire Line
-	7200 3650 7200 4000
-Connection ~ 6650 3650
-Wire Wire Line
-	6650 3650 6650 4000
-$Comp
-L RC1206JR-07110RL:RC1206JR-07110RL R7
-U 1 1 6156637C
-P 7200 4800
-F 0 "R7" V 7154 4905 50  0000 L CNN
-F 1 "RC1206JR-07110RL" V 7245 4905 50  0000 L CNN
-F 2 "RESC3116X65N" H 7200 4800 50  0001 L BNN
-F 3 "" H 7200 4800 50  0001 L BNN
-	1    7200 4800
-	0    1    1    0
-$EndComp
-Entry Wire Line
-	3850 4200 3950 4300
-Wire Wire Line
-	3950 4300 3950 5450
-Wire Wire Line
-	3950 5450 7200 5450
-Text Label 3950 4550 0    50   ~ 0
-GPIO22
 $Comp
 L 1825255-1:1825255-1 S1
@@
 $EndComp
 Wire Wire Line
-	7200 5450 7200 5200
-Wire Wire Line
-	4950 4150 5400 4150
-Wire Wire Line
 	6150 4000 6150 3850
 Wire Wire Line
@@
 	5400 3850 5400 4050
 NoConn ~ 5400 4250
-Wire Bus Line
-	3850 3900 3850 4350
 Text HLabel 3650 3900 0    50   BiDi ~ 0
 TIME_OF_USE_DATA
+Wire Wire Line
+	3950 4150 5400 4150
+Wire Wire Line
+	6650 3500 6650 4000
+Wire Bus Line
+	3850 3900 3850 4050
 $EndSCHEMATC

Commit message: udpated circuit
Parts:
- added R?: RMCF1206JT150R, RESC3216X70N, symbol RMCF1206JT150R:RMCF1206JT150R
Connections:
- net GPIO17: now also R?.1
- new net GND: R?.2
Changed lines of the file:
@@
 TIME_OF_USE_DATA
 Wire Wire Line
-	3950 4150 5400 4150
+	3950 4150 4650 4150
 Wire Wire Line
 	6650 3500 6650 4000
 Wire Bus Line
 	3850 3900 3850 4050
+$Comp
+L RMCF1206JT150R:RMCF1206JT150R R?
+U 1 1 61705C6B
+P 4650 4550
+F 0 "R?" V 4604 4655 50  0000 L CNN
+F 1 "RMCF1206JT150R" V 4695 4655 50  0000 L CNN
+F 2 "RESC3216X70N" H 4650 4550 50  0001 L BNN
+F 3 "" H 4650 4550 50  0001 L BNN
+	1    4650 4550
+	0    1    1    0
+$EndComp
+Connection ~ 4650 4150
+Wire Wire Line
+	4650 4150 5400 4150
+$Comp
+L power:GND #PWR?
+U 1 1 61707039
+P 4650 4950
+F 0 "#PWR?" H 4650 4700 50  0001 C CNN
+F 1 "GND" H 4655 4777 50  0000 C CNN
+F 2 "" H 4650 4950 50  0001 C CNN
+F 3 "" H 4650 4950 50  0001 C CNN
+	1    4650 4950
+	1    0    0    -1
+$EndComp
 $EndSCHEMATC

Commit message: schematic updates
Parts:
- removed R?: RMCF1206JT150R, RESC3216X70N, symbol RMCF1206JT150R:RMCF1206JT150R
- added R7: 10k, RESC3115X60N, symbol RNCP1206FTD10K0:RNCP1206FTD10K0
Connections:
- net GND: now also R7.2
- net at S1.3: now also R7.1
- net +5V renamed +3V3
- net GPIO17 renamed GPIO22
- no-connect marks 1 -> 0
Changed lines of the file:
@@
 Comment4 ""
 $EndDescr
-$Comp
-L power:+5V #PWR07
-U 1 1 614A5231
-P 6650 3500
-F 0 "#PWR07" H 6650 3350 50  0001 C CNN
-F 1 "+5V" H 6665 3673 50  0000 C CNN
-F 2 "" H 6650 3500 50  0001 C CNN
-F 3 "" H 6650 3500 50  0001 C CNN
-	1    6650 3500
-	1    0    0    -1
-$EndComp
 Wire Wire Line
 	6650 4000 6150 4000
-Text Label 4150 4150 0    50   ~ 0
-GPIO17
-Entry Wire Line
-	3850 4050 3950 4150
-Wire Bus Line
-	3650 3900 3850 3900
 $Comp
 L 1825255-1:1825255-1 S1
@@
 Wire Wire Line
 	5400 3850 5400 4050
-NoConn ~ 5400 4250
+Wire Wire Line
+	6650 3500 6650 4000
+$Comp
+L power:GND #PWR07
+U 1 1 61707039
+P 4900 5050
+F 0 "#PWR07" H 4900 4800 50  0001 C CNN
+F 1 "GND" H 4905 4877 50  0000 C CNN
+F 2 "" H 4900 5050 50  0001 C CNN
+F 3 "" H 4900 5050 50  0001 C CNN
+	1    4900 5050
+	1    0    0    -1
+$EndComp
+$Comp
+L power:+3.3V #PWR08
+U 1 1 6174D417
+P 6650 3500
+F 0 "#PWR08" H 6650 3350 50  0001 C CNN
+F 1 "+3.3V" H 6665 3673 50  0000 C CNN
+F 2 "" H 6650 3500 50  0001 C CNN
+F 3 "" H 6650 3500 50  0001 C CNN
+	1    6650 3500
+	1    0    0    -1
+$EndComp
+Wire Wire Line
+	3950 4150 5400 4150
+Wire Bus Line
+	3850 3900 3850 4050
 Text HLabel 3650 3900 0    50   BiDi ~ 0
 TIME_OF_USE_DATA
+Wire Bus Line
+	3650 3900 3850 3900
+Entry Wire Line
+	3850 4050 3950 4150
+Text Label 4150 4150 0    50   ~ 0
+GPIO22
 Wire Wire Line
-	3950 4150 4650 4150
-Wire Wire Line
-	6650 3500 6650 4000
-Wire Bus Line
-	3850 3900 3850 4050
+	4900 4250 5400 4250
 $Comp
-L RMCF1206JT150R:RMCF1206JT150R R?
-U 1 1 61705C6B
-P 4650 4550
-F 0 "R?" V 4604 4655 50  0000 L CNN
-F 1 "RMCF1206JT150R" V 4695 4655 50  0000 L CNN
-F 2 "RESC3216X70N" H 4650 4550 50  0001 L BNN
-F 3 "" H 4650 4550 50  0001 L BNN
-	1    4650 4550
+L RNCP1206FTD10K0:RNCP1206FTD10K0 R7
+U 1 1 617867AC
+P 4900 4650
+F 0 "R7" V 4854 4755 50  0000 L CNN
+F 1 "10k" V 4945 4755 50  0000 L CNN
+F 2 "RESC3115X60N" H 4900 4650 50  0001 L BNN
+F 3 "" H 4900 4650 50  0001 L BNN
+	1    4900 4650
 	0    1    1    0
 $EndComp
-Connection ~ 4650 4150
-Wire Wire Line
-	4650 4150 5400 4150
-$Comp
-L power:GND #PWR?
-U 1 1 61707039
-P 4650 4950
-F 0 "#PWR?" H 4650 4700 50  0001 C CNN
-F 1 "GND" H 4655 4777 50  0000 C CNN
-F 2 "" H 4650 4950 50  0001 C CNN
-F 3 "" H 4650 4950 50  0001 C CNN
-	1    4650 4950
-	1    0    0    -1
-$EndComp
 $EndSCHEMATC

Commit message: PCB changes
Parts:
- R6: renamed from R7; footprint RESC3115X60N -> RNCP1206FTD10K0:RESC3115X60N
- S1: footprint SW_1825255-1 -> 1825255-1:SW_1825255-1
Changed lines of the file:
@@
 F 0 "S1" H 6030 4296 50  0000 L CNN
 F 1 "1825255-1" H 6030 4205 50  0000 L CNN
-F 2 "SW_1825255-1" H 5800 4250 50  0001 L BNN
+F 2 "1825255-1:SW_1825255-1" H 5800 4250 50  0001 L BNN
 F 3 "" H 5800 4250 50  0001 L BNN
 F 4 "1825255-1" H 5800 4250 50  0001 L BNN "Comment"
@@
 	4900 4250 5400 4250
 $Comp
-L RNCP1206FTD10K0:RNCP1206FTD10K0 R7
+L RNCP1206FTD10K0:RNCP1206FTD10K0 R6
 U 1 1 617867AC
 P 4900 4650
-F 0 "R7" V 4854 4755 50  0000 L CNN
+F 0 "R6" V 4854 4755 50  0000 L CNN
 F 1 "10k" V 4945 4755 50  0000 L CNN
-F 2 "RESC3115X60N" H 4900 4650 50  0001 L BNN
+F 2 "RNCP1206FTD10K0:RESC3115X60N" H 4900 4650 50  0001 L BNN
 F 3 "" H 4900 4650 50  0001 L BNN
 	1    4900 4650
