File: Hardware/tool_circuit/Time_of_Use.sch (KiCad schematic (older format))
At the start: 1 part, among them SW1 Switch

Commit message: pulling
Connections:
- net GPIO22_GEN3 renamed Time_of_use
Changed lines of the file:
@@
 	5650 3500 5650 4300
 Text GLabel 8350 3850 2    50   BiDi ~ 0
-GPIO22_GEN3
+Time_of_use
 $Comp
 L power:+3.3V #PWR0101
