File: Hardware/tool_circuit/raspberrypi_header.sch (KiCad schematic (older format))
At the start: 5 parts, among them J4 GPIO_CONNECTOR

Commit message: schematic LEDs + switch
Parts:
- added D1: 5BC-3-CA-F, 3_PIN_CONNECTOR, symbol 5BC-3-CA-F:5BC-3-CA-F
- added D2: WP7113YD, LED_WP7113YD, symbol WP7113YD:WP7113YD
- added R10: ERJ1TNF30R9U, RES_ERJ1TNF30R9U, symbol ERJ1TNF30R9U:ERJ1TNF30R9U
- added R11, R9: SLI-343M8C3F, LED_SLI-343D_ROM, symbol 2021-09-28_17-40-03:SLI-343M8C3F
- added R12: RMCF1206FT140R, RES_RMCF1206_STP, symbol 2021-09-28_17-48-03:RMCF1206FT140R
- added R13: S2-100RF1, RES_S2-2615_6P6X3P9_RDN, symbol 2021-09-28_16-21-53:S2-100RF1
- added R8: ERJ8ENF54R9V, RES_ERJ8ENF54R9V, symbol ERJ8ENF54R9V:ERJ8ENF54R9V
Connections:
- net labels added: 3.3V_LED, 5V_LED, Data_Transfer, Enable_Disable, GPIO17, GPIO2, GPIO22, GPIO27, GPIO3
- wire segments 57 -> 69
Other:
- moved on the sheet: H1, H2, H3, H4

Commit message: made some post review changes
Connections:
- net labels added: PI_CONN
- no-connect marks 28 -> 21
Changed lines of the file:
@@
 Wire Wire Line
 	6200 1950 6200 2050
-Text Label 4100 2150 0    50   ~ 0
-GPIO2_SDA1
-Text Label 4100 2250 0    50   ~ 0
-GPIO3_SCL1
 Text Label 4100 2350 0    50   ~ 0
 GPIO4_GPIO_GCLK
-Text Label 4100 2550 0    50   ~ 0
-GPIO17_GEN0
-Text Label 4100 2650 0    50   ~ 0
-GPIO27_GEN2
-Text Label 4100 2750 0    50   ~ 0
-GPIO22_GEN3
 Text Label 4100 2950 0    50   ~ 0
 GPIO10_SPI_MOSI
@@
 Text Label 4100 3850 0    50   ~ 0
 GPIO26
-NoConn ~ 4000 2150
-NoConn ~ 4000 2250
 NoConn ~ 4000 2350
-NoConn ~ 4000 2550
-NoConn ~ 4000 2650
-NoConn ~ 4000 2750
 NoConn ~ 4000 2950
 NoConn ~ 4000 3050
@@
 NoConn ~ 6600 2450
 NoConn ~ 6600 2550
-NoConn ~ 6600 2750
-NoConn ~ 6600 2850
 NoConn ~ 6600 3050
 NoConn ~ 6600 3150
@@
 Wire Wire Line
 	3150 2750 5050 2750
+Text Label 3300 2750 0    50   ~ 0
+GPIO22
+Text HLabel 2350 1950 0    50   BiDi ~ 0
+PI_CONN
+Text Label 4100 2150 0    50   ~ 0
+GPIO2_SDA1
+Text Label 4100 2250 0    50   ~ 0
+GPIO3_SCL1
+Text Label 4100 2550 0    50   ~ 0
+GPIO17_GEN0
+Text Label 4100 2750 0    50   ~ 0
+GPIO22_GEN3
+Text Label 4100 2650 0    50   ~ 0
+GPIO27_GEN2
 Wire Bus Line
 	3050 1950 3050 2800
-Text Label 3300 2750 0    50   ~ 0
-GPIO22
 $EndSCHEMATC

Commit message: Latest revisions to schematic
Parts:
- removed D1: 5BC-3-CA-F, 3_PIN_CONNECTOR, symbol 5BC-3-CA-F:5BC-3-CA-F
- removed R10: ERJ1TNF30R9U, RES_ERJ1TNF30R9U, symbol ERJ1TNF30R9U:ERJ1TNF30R9U
- removed R12: RMCF1206FT140R, RES_RMCF1206_STP, symbol 2021-09-28_17-48-03:RMCF1206FT140R
- removed R13: S2-100RF1, RES_S2-2615_6P6X3P9_RDN, symbol 2021-09-28_16-21-53:S2-100RF1
- removed R8: ERJ8ENF54R9V, RES_ERJ8ENF54R9V, symbol ERJ8ENF54R9V:ERJ8ENF54R9V
- added D?: WL-TMRC, symbol WL-TMRC:WL-TMRC
- added LED?: 151034BS03000, LED_BS03000_WRE, symbol 2021-09-28_17-07-40:151034BS03000
- added R?: SLI-343M8C3F, LED_SLI-343D_ROM, symbol 2021-09-28_17-40-03:SLI-343M8C3F
- added R? (x3): 100, RESC3115X60N, symbol RNCP1206FTD100R:RNCP1206FTD100R
- added R?: 130, RESC3116X65N, symbol AC1206FR-07130RL:AC1206FR-07130RL
- added R?: 42.2, RESC3116X65N, symbol RC1206FR-0742R2L:RC1206FR-0742R2L
- added R?: 220, RESC3216X70N, symbol RMCF1206JT220R:RMCF1206JT220R
- added TP? (x6): S2751-46R, HARWIN_S2751-46R, symbol S2751-46R:S2751-46R
Connections:
- net labels added: Disable_LED, Enable_LED, Tool_In_Use
- net labels removed: Enable_Disable, GPIO22
- wire segments 69 -> 68
- no-connect marks 21 -> 20
Other:
- moved on the sheet: D2

Commit message: schematic updates
Parts:
- gave numbers to parts that had none: 15
- renumbered R11 to R15
Connections:
- net labels removed: GPIO17
- wire segments 68 -> 69
- no-connect marks 20 -> 21
Changed lines of the file:
@@
 $EndComp
 $Comp
-L power:GND #PWR014
+L power:GND #PWR016
 U 1 1 5C777805
 P 4850 4100
-F 0 "#PWR014" H 4850 3850 50  0001 C CNN
+F 0 "#PWR016" H 4850 3850 50  0001 C CNN
 F 1 "GND" H 4855 3927 50  0001 C CNN
 F 2 "" H 4850 4100 50  0001 C CNN
@@
 $EndComp
 $Comp
-L power:GND #PWR015
+L power:GND #PWR017
 U 1 1 5C777838
 P 5750 4100
-F 0 "#PWR015" H 5750 3850 50  0001 C CNN
+F 0 "#PWR017" H 5750 3850 50  0001 C CNN
 F 1 "GND" H 5755 3927 50  0001 C CNN
 F 2 "" H 5750 4100 50  0001 C CNN
@@
 	5750 3650 5750 4100
 $Comp
-L power:+3.3V #PWR013
+L power:+3.3V #PWR015
 U 1 1 5C777AB0
 P 4800 1950
-F 0 "#PWR013" H 4800 1800 50  0001 C CNN
+F 0 "#PWR015" H 4800 1800 50  0001 C CNN
 F 1 "+3.3V" H 4815 2123 50  0000 C CNN
 F 2 "" H 4800 1950 50  0001 C CNN
@@
 Connection ~ 4800 2050
 $Comp
-L power:+5V #PWR016
+L power:+5V #PWR018
 U 1 1 5C777E01
 P 5850 1950
-F 0 "#PWR016" H 5850 1800 50  0001 C CNN
+F 0 "#PWR018" H 5850 1800 50  0001 C CNN
 F 1 "+5V" H 5865 2123 50  0000 C CNN
 F 2 "" H 5850 1950 50  0001 C CNN
@@
 Wire Wire Line
 	5850 2050 5850 1950
-Wire Wire Line
-	5550 2150 5850 2150
-Wire Wire Line
-	5850 2150 5850 2050
 Connection ~ 5850 2050
-$Comp
-L power:GND #PWR012
-U 1 1 5C778504
-P 4450 4200
-F 0 "#PWR012" H 4450 3950 50  0001 C CNN
-F 1 "GND" H 4455 4027 50  0001 C CNN
-F 2 "" H 4450 4200 50  0001 C CNN
-F 3 "" H 4450 4200 50  0001 C CNN
-	1    4450 4200
-	1    0    0    -1
-$EndComp
-$Comp
-L power:PWR_FLAG #FLG02
-U 1 1 5C778511
-P 4450 4150
-F 0 "#FLG02" H 4450 4225 50  0001 C CNN
-F 1 "PWR_FLAG" H 4450 4324 50  0000 C CNN
-F 2 "" H 4450 4150 50  0001 C CNN
-F 3 "~" H 4450 4150 50  0001 C CNN
-	1    4450 4150
-	1    0    0    -1
-$EndComp
-Wire Wire Line
-	4450 4150 4450 4200
 Text Notes 7100 1100 0    50   ~ 10
 If back powering Pi with 5V \nNOTE that the Raspberry Pi 3B+ and Pi Zero \nand ZeroW do not include an input ZVD.
@@
 	1    0    0    -1
 $EndComp
-Wire Bus Line
-	2350 1950 3050 1950
-Entry Wire Line
-	3050 2050 3150 2150
-Entry Wire Line
-	3050 2150 3150 2250
-Entry Wire Line
-	3050 2450 3150 2550
-Entry Wire Line
-	3050 2550 3150 2650
-Wire Wire Line
-	3150 2150 5050 2150
-Wire Wire Line
-	3150 2250 5050 2250
-Wire Wire Line
-	3150 2550 5050 2550
-Wire Wire Line
-	3150 2650 5050 2650
+Wire Wire Line
+	2050 2150 5050 2150
 Text Label 3250 2150 0    50   ~ 0
 GPIO2
 Text Label 3250 2250 0    50   ~ 0
 GPIO3
-Text Label 3300 2650 0    50   ~ 0
-GPIO27
-Text Label 3300 2550 0    50   ~ 0
-GPIO17
 $Comp
 L WP7113YD:WP7113YD D2
@@
 	8100 2750 8100 2800
 $Comp
-L power:GND #PWR0103
+L power:GND #PWR019
 U 1 1 61539C99
 P 7100 4450
-F 0 "#PWR0103" H 7100 4200 50  0001 C CNN
+F 0 "#PWR019" H 7100 4200 50  0001 C CNN
 F 1 "GND" H 7105 4277 50  0000 C CNN
 F 2 "" H 7100 4450 50  0001 C CNN
@@
 	5550 2850 7300 2850
 $Comp
-L power:GND #PWR0104
+L power:GND #PWR020
 U 1 1 6155009E
 P 7450 4150
-F 0 "#PWR0104" H 7450 3900 50  0001 C CNN
+F 0 "#PWR020" H 7450 3900 50  0001 C CNN
 F 1 "GND" H 7455 3977 50  0000 C CNN
 F 2 "" H 7450 4150 50  0001 C CNN
@@
 Enable_LED
 $Comp
-L 2021-09-28_17-40-03:SLI-343M8C3F R11
+L 2021-09-28_17-40-03:SLI-343M8C3F R15
 U 1 1 61576EA3
 P 7900 2000
-F 0 "R11" H 8100 2388 60  0000 C CNN
+F 0 "R15" H 8100 2388 60  0000 C CNN
 F 1 "SLI-343M8C3F" H 8100 2282 60  0000 C CNN
 F 2 "LED_SLI-343D_ROM" H 8100 1640 60  0001 C CNN
@@
 Wire Wire Line
 	7000 2150 7000 2000
-Connection ~ 5850 2150
 Text Label 6700 2150 0    50   ~ 0
 5V_LED
 Connection ~ 4800 2850
 $Comp
-L power:GND #PWR0105
+L power:GND #PWR022
 U 1 1 6157F3DC
 P 8300 2000
-F 0 "#PWR0105" H 8300 1750 50  0001 C CNN
+F 0 "#PWR022" H 8300 1750 50  0001 C CNN
 F 1 "GND" V 8305 1872 50  0000 R CNN
 F 2 "" H 8300 2000 50  0001 C CNN
@@
 	3300 2850 3600 2850
 $Comp
-L power:GND #PWR0106
+L power:GND #PWR014
 U 1 1 61585D7E
 P 3300 4250
-F 0 "#PWR0106" H 3300 4000 50  0001 C CNN
+F 0 "#PWR014" H 3300 4000 50  0001 C CNN
 F 1 "GND" H 3305 4077 50  0000 C CNN
 F 2 "" H 3300 4250 50  0001 C CNN
@@
 Text Label 2850 2750 0    50   ~ 0
 Tool_In_Use
-Text HLabel 2350 1950 0    50   BiDi ~ 0
-PI_CONN
 Text Label 4100 2150 0    50   ~ 0
 GPIO2_SDA1
@@
 GPIO27_GEN2
 $Comp
-L 2021-09-28_17-40-03:SLI-343M8C3F R?
+L 2021-09-28_17-40-03:SLI-343M8C3F R12
 U 1 1 6161302E
 P 7450 2950
-F 0 "R?" H 7650 3338 60  0000 C CNN
+F 0 "R12" H 7650 3338 60  0000 C CNN
 F 1 "SLI-343M8C3F" H 7650 3232 60  0000 C CNN
 F 2 "LED_SLI-343D_ROM" H 7650 2590 60  0001 C CNN
@@
 $EndComp
 $Comp
-L WL-TMRC:WL-TMRC D?
+L WL-TMRC:WL-TMRC D1
 U 1 1 6161A01D
 P 7100 3450
-F 0 "D?" V 7168 3311 50  0000 R CNN
+F 0 "D1" V 7168 3311 50  0000 R CNN
 F 1 "WL-TMRC" V 7077 3311 50  0000 R CNN
 F 2 "" H 7100 3450 50  0001 C CNN
@@
 	5550 3050 6900 3050
 $Comp
-L RNCP1206FTD100R:RNCP1206FTD100R R?
+L RNCP1206FTD100R:RNCP1206FTD100R R11
 U 1 1 61624927
 P 7100 4050
-F 0 "R?" V 7054 4155 50  0000 L CNN
+F 0 "R11" V 7054 4155 50  0000 L CNN
 F 1 "100" V 7145 4155 50  0000 L CNN
 F 2 "RESC3115X60N" H 7100 4050 50  0001 L BNN
@@
 $EndComp
 $Comp
-L RNCP1206FTD100R:RNCP1206FTD100R R?
+L RNCP1206FTD100R:RNCP1206FTD100R R13
 U 1 1 616261C1
 P 7450 3750
-F 0 "R?" V 7404 3855 50  0000 L CNN
+F 0 "R13" V 7404 3855 50  0000 L CNN
 F 1 "100" V 7495 3855 50  0000 L CNN
 F 2 "RESC3115X60N" H 7450 3750 50  0001 L BNN
@@
 $EndComp
 $Comp
-L RNCP1206FTD100R:RNCP1206FTD100R R?
+L RNCP1206FTD100R:RNCP1206FTD100R R10
 U 1 1 61626B9B
 P 3300 3850
-F 0 "R?" V 3254 3955 50  0000 L CNN
+F 0 "R10" V 3254 3955 50  0000 L CNN
 F 1 "100" V 3345 3955 50  0000 L CNN
 F 2 "RESC3115X60N" H 3300 3850 50  0001 L BNN
@@
 P 2050 3300
 AR Path="/611DF2F9/61630B5E" Ref="LED?"  Part="1"
-AR Path="/61514F71/61630B5E" Ref="LED?"  Part="1"
-F 0 "LED?" V 2197 3528 60  0000 L CNN
+AR Path="/61514F71/61630B5E" Ref="LED1"  Part="1"
+F 0 "LED1" V 2197 3528 60  0000 L CNN
 F 1 "151034BS03000" V 2303 3528 60  0000 L CNN
 F 2 "LED_BS03000_WRE" H 2250 2940 60  0001 C CNN
@@
 P 2050 4500
 AR Path="/611DF2F9/61630B6B" Ref="#PWR?"  Part="1"
-AR Path="/61514F71/61630B6B" Ref="#PWR?"  Part="1"
-F 0 "#PWR?" H 2050 4250 50  0001 C CNN
+AR Path="/61514F71/61630B6B" Ref="#PWR013"  Part="1"
+F 0 "#PWR013" H 2050 4250 50  0001 C CNN
 F 1 "GND" H 2055 4327 50  0000 C CNN
 F 2 "" H 2050 4500 50  0001 C CNN
@@
 	2050 2750 2350 2750
 $Comp
-L S2751-46R:S2751-46R TP?
+L S2751-46R:S2751-46R TP5
 U 1 1 61650FDF
 P 4950 1950
-F 0 "TP?" H 5035 2017 50  0000 L CNN
+F 0 "TP5" H 5035 2017 50  0000 L CNN
 F 1 "S2751-46R" H 5035 1926 50  0000 L CNN
 F 2 "HARWIN_S2751-46R" H 4950 1950 50  0001 L BNN
@@
 	4950 2050 5050 2050
 $Comp
-L S2751-46R:S2751-46R TP?
+L S2751-46R:S2751-46R TP8
 U 1 1 61651CC8
 P 7450 2650
-F 0 "TP?" H 7535 2717 50  0000 L CNN
+F 0 "TP8" H 7535 2717 50  0000 L CNN
 F 1 "S2751-46R" H 7535 2626 50  0000 L CNN
 F 2 "HARWIN_S2751-46R" H 7450 2650 50  0001 L BNN
@@
 	7450 2750 8100 2750
 $Comp
-L S2751-46R:S2751-46R TP?
+L S2751-46R:S2751-46R TP7
 U 1 1 6165274B
 P 7300 2950
-F 0 "TP?" H 7215 2924 50  0000 R CNN
+F 0 "TP7" H 7215 2924 50  0000 R CNN
 F 1 "S2751-46R" H 7215 3015 50  0000 R CNN
 F 2 "HARWIN_S2751-46R" H 7300 2950 50  0001 L BNN
@@
 	7300 2850 7450 2850
 $Comp
-L S2751-46R:S2751-46R TP?
+L S2751-46R:S2751-46R TP6
 U 1 1 61653544
 P 6900 3150
-F 0 "TP?" H 6815 3124 50  0000 R CNN
+F 0 "TP6" H 6815 3124 50  0000 R CNN
 F 1 "S2751-46R" H 6815 3215 50  0000 R CNN
 F 2 "HARWIN_S2751-46R" H 6900 3150 50  0001 L BNN
@@
 	6900 3050 7100 3050
 $Comp
-L S2751-46R:S2751-46R TP?
+L S2751-46R:S2751-46R TP4
 U 1 1 61653BD5
 P 3600 2950
-F 0 "TP?" H 3515 2924 50  0000 R CNN
+F 0 "TP4" H 3515 2924 50  0000 R CNN
 F 1 "S2751-46R" H 3515 3015 50  0000 R CNN
 F 2 "HARWIN_S2751-46R" H 3600 2950 50  0001 L BNN
@@
 	3600 2850 4800 2850
 $Comp
-L S2751-46R:S2751-46R TP?
+L S2751-46R:S2751-46R TP3
 U 1 1 61654750
 P 2350 2850
-F 0 "TP?" H 2265 2824 50  0000 R CNN
+F 0 "TP3" H 2265 2824 50  0000 R CNN
 F 1 "S2751-46R" H 2265 2915 50  0000 R CNN
 F 2 "HARWIN_S2751-46R" H 2350 2850 50  0001 L BNN
@@
 	-1   0    0    1
 $EndComp
-Connection ~ 2350 2750
 Wire Wire Line
 	2350 2750 5050 2750
 $Comp
-L AC1206FR-07130RL:AC1206FR-07130RL R?
+L AC1206FR-07130RL:AC1206FR-07130RL R16
 U 1 1 61659CB7
 P 8100 3900
-F 0 "R?" V 8054 4005 50  0000 L CNN
+F 0 "R16" V 8054 4005 50  0000 L CNN
 F 1 "130" V 8145 4005 50  0000 L CNN
 F 2 "RESC3116X65N" H 8100 3900 50  0001 L BNN
@@
 $EndComp
 $Comp
-L power:GND #PWR?
+L power:GND #PWR021
 U 1 1 6165AE6F
 P 8100 4300
-F 0 "#PWR?" H 8100 4050 50  0001 C CNN
+F 0 "#PWR021" H 8100 4050 50  0001 C CNN
 F 1 "GND" H 8105 4127 50  0000 C CNN
 F 2 "" H 8100 4300 50  0001 C CNN
@@
 $EndComp
 $Comp
-L RC1206FR-0742R2L:RC1206FR-0742R2L R?
+L RC1206FR-0742R2L:RC1206FR-0742R2L R8
 U 1 1 6165D04D
 P 2050 4100
-F 0 "R?" V 2004 4205 50  0000 L CNN
+F 0 "R8" V 2004 4205 50  0000 L CNN
 F 1 "42.2" V 2095 4205 50  0000 L CNN
 F 2 "RESC3116X65N" H 2050 4100 50  0001 L BNN
@@
 	3300 2850 3300 3050
 $Comp
-L RMCF1206JT220R:RMCF1206JT220R R?
+L RMCF1206JT220R:RMCF1206JT220R R14
 U 1 1 61665485
 P 7500 2000
-F 0 "R?" H 7500 2242 50  0000 C CNN
+F 0 "R14" H 7500 2242 50  0000 C CNN
 F 1 "220" H 7500 2151 50  0000 C CNN
 F 2 "RESC3216X70N" H 7500 2000 50  0001 L BNN
@@
 	1    0    0    -1
 $EndComp
+Connection ~ 2350 2750
+Connection ~ 5850 2150
+Wire Wire Line
+	5850 2150 5850 2050
+Wire Wire Line
+	5550 2150 5850 2150
+Text Label 3300 2650 0    50   ~ 0
+GPIO27
+Entry Wire Line
+	1950 2650 2050 2750
+Text HLabel 1250 2050 0    50   BiDi ~ 0
+PI_CONN
+Entry Wire Line
+	1950 2550 2050 2650
+Entry Wire Line
+	1950 2250 2050 2350
+Entry Wire Line
+	1950 2050 2050 2150
 Wire Bus Line
-	3050 1950 3050 2550
+	1250 2050 1950 2050
+Wire Wire Line
+	5050 2250 2200 2250
+Wire Wire Line
+	2200 2250 2200 2350
+Wire Wire Line
+	2200 2350 2050 2350
+Wire Wire Line
+	2050 2650 5050 2650
+Wire Wire Line
+	5050 2550 4050 2550
+NoConn ~ 4050 2550
+Wire Bus Line
+	1950 2050 1950 2650
 $EndSCHEMATC

Commit message: PCB changes
Parts:
- removed R10, R11, R13: 100, RESC3115X60N, symbol RNCP1206FTD100R:RNCP1206FTD100R
- removed R12, R15, R9: SLI-343M8C3F, LED_SLI-343D_ROM, symbol 2021-09-28_17-40-03:SLI-343M8C3F
- added D2, D4, D6: Green, WP7113GD:LED_WP7113GD, symbol WP7113GD:WP7113GD
- added R10, R8, R9: 100, footprints:RNCP1206FTD100R, symbol 2021-10-29_06-40-06:RNCP1206FTD100R
- D3: renamed from D1; value WL-TMRC -> Red; footprint (none) -> WL-TMRC:LED-5MM-ROUND
- D5: renamed from D2; value WP7113YD -> Yellow; footprint LED_WP7113YD -> WP7113YD:LED_WP7113YD
- LED1: value 151034BS03000 -> Blue; footprint LED_BS03000_WRE -> Blue LED:151034BS03000
- R11: renamed from R14; footprint RESC3216X70N -> RMCF1206JT220R:RESC3216X70N
- R12: renamed from R16; footprint RESC3116X65N -> AC1206FR-07130RL:RESC3116X65N
- R7: renamed from R8; footprint RESC3116X65N -> RC1206FR-0742R2L:RESC3116X65N
- TP3, TP4, TP5, TP6, TP7, TP8: footprint HARWIN_S2751-46R -> S2751-46R:HARWIN_S2751-46R
Connections:
- wire segments 69 -> 70

Commit message: layout
Parts:
- renumbered D2 to D1, D3 to D2, D4 to D3, D5 to D4, D6 to D5, R7 to R2, R8 to R3, R9 to R4, R10 to R5, R11 to R6, R12 to R7
Changed lines of the file:
@@
 $EndComp
 $Comp
-L power:GND #PWR016
+L power:GND #PWR015
 U 1 1 5C777805
 P 4850 4100
-F 0 "#PWR016" H 4850 3850 50  0001 C CNN
+F 0 "#PWR015" H 4850 3850 50  0001 C CNN
 F 1 "GND" H 4855 3927 50  0001 C CNN
 F 2 "" H 4850 4100 50  0001 C CNN
@@
 $EndComp
 $Comp
-L power:GND #PWR017
+L power:GND #PWR016
 U 1 1 5C777838
 P 5750 4100
-F 0 "#PWR017" H 5750 3850 50  0001 C CNN
+F 0 "#PWR016" H 5750 3850 50  0001 C CNN
 F 1 "GND" H 5755 3927 50  0001 C CNN
 F 2 "" H 5750 4100 50  0001 C CNN
@@
 	5750 3650 5750 4100
 $Comp
-L power:+3.3V #PWR015
+L power:+3.3V #PWR014
 U 1 1 5C777AB0
 P 4800 1950
-F 0 "#PWR015" H 4800 1800 50  0001 C CNN
+F 0 "#PWR014" H 4800 1800 50  0001 C CNN
 F 1 "+3.3V" H 4815 2123 50  0000 C CNN
 F 2 "" H 4800 1950 50  0001 C CNN
@@
 Connection ~ 4800 2050
 $Comp
-L power:+5V #PWR018
+L power:+5V #PWR017
 U 1 1 5C777E01
 P 5850 1950
-F 0 "#PWR018" H 5850 1800 50  0001 C CNN
+F 0 "#PWR017" H 5850 1800 50  0001 C CNN
 F 1 "+5V" H 5865 2123 50  0000 C CNN
 F 2 "" H 5850 1950 50  0001 C CNN
@@
 Wire Wire Line
 	5550 2050 5850 2050
-Wire Wire Line
-	5850 2050 5850 1950
-Connection ~ 5850 2050
 Text Notes 7100 1100 0    50   ~ 10
 If back powering Pi with 5V \nNOTE that the Raspberry Pi 3B+ and Pi Zero \nand ZeroW do not include an input ZVD.
@@
 GPIO3
 $Comp
-L WP7113YD:WP7113YD D5
+L WP7113YD:WP7113YD D4
 U 1 1 61534E0C
 P 8100 3200
-F 0 "D5" V 8196 3121 50  0000 R CNN
+F 0 "D4" V 8196 3121 50  0000 R CNN
 F 1 "Yellow" V 8105 3121 50  0000 R CNN
 F 2 "WP7113YD:LED_WP7113YD" H 8100 3200 50  0001 L BNN
@@
 	8100 2750 8100 2800
 $Comp
-L power:GND #PWR019
+L power:GND #PWR018
 U 1 1 61539C99
 P 7100 4150
-F 0 "#PWR019" H 7100 3900 50  0001 C CNN
+F 0 "#PWR018" H 7100 3900 50  0001 C CNN
 F 1 "GND" H 7105 3977 50  0000 C CNN
 F 2 "" H 7100 4150 50  0001 C CNN
@@
 	5550 2850 7300 2850
 $Comp
-L power:GND #PWR020
+L power:GND #PWR019
 U 1 1 6155009E
 P 7450 4150
-F 0 "#PWR020" H 7450 3900 50  0001 C CNN
+F 0 "#PWR019" H 7450 3900 50  0001 C CNN
 F 1 "GND" H 7455 3977 50  0000 C CNN
 F 2 "" H 7450 4150 50  0001 C CNN
@@
 Connection ~ 4800 2850
 $Comp
-L power:GND #PWR022
+L power:GND #PWR021
 U 1 1 6157F3DC
 P 8800 2000
-F 0 "#PWR022" H 8800 1750 50  0001 C CNN
+F 0 "#PWR021" H 8800 1750 50  0001 C CNN
 F 1 "GND" V 8805 1872 50  0000 R CNN
 F 2 "" H 8800 2000 50  0001 C CNN
@@
 	3300 2850 3600 2850
 $Comp
-L power:GND #PWR014
+L power:GND #PWR013
 U 1 1 61585D7E
 P 3300 4250
-F 0 "#PWR014" H 3300 4000 50  0001 C CNN
+F 0 "#PWR013" H 3300 4000 50  0001 C CNN
 F 1 "GND" H 3305 4077 50  0000 C CNN
 F 2 "" H 3300 4250 50  0001 C CNN
@@
 P 2050 4500
 AR Path="/611DF2F9/61630B6B" Ref="#PWR?"  Part="1"
-AR Path="/61514F71/61630B6B" Ref="#PWR013"  Part="1"
-F 0 "#PWR013" H 2050 4250 50  0001 C CNN
+AR Path="/61514F71/61630B6B" Ref="#PWR012"  Part="1"
+F 0 "#PWR012" H 2050 4250 50  0001 C CNN
 F 1 "GND" H 2055 4327 50  0000 C CNN
 F 2 "" H 2050 4500 50  0001 C CNN
@@
 	2350 2750 5050 2750
 $Comp
-L AC1206FR-07130RL:AC1206FR-07130RL R12
+L AC1206FR-07130RL:AC1206FR-07130RL R7
 U 1 1 61659CB7
 P 8100 3900
-F 0 "R12" V 8054 4005 50  0000 L CNN
+F 0 "R7" V 8054 4005 50  0000 L CNN
 F 1 "130" V 8145 4005 50  0000 L CNN
 F 2 "AC1206FR-07130RL:RESC3116X65N" H 8100 3900 50  0001 L BNN
@@
 $EndComp
 $Comp
-L power:GND #PWR021
+L power:GND #PWR020
 U 1 1 6165AE6F
 P 8100 4300
-F 0 "#PWR021" H 8100 4050 50  0001 C CNN
+F 0 "#PWR020" H 8100 4050 50  0001 C CNN
 F 1 "GND" H 8105 4127 50  0000 C CNN
 F 2 "" H 8100 4300 50  0001 C CNN
@@
 $EndComp
 $Comp
-L RC1206FR-0742R2L:RC1206FR-0742R2L R7
+L RC1206FR-0742R2L:RC1206FR-0742R2L R2
 U 1 1 6165D04D
 P 2050 4100
-F 0 "R7" V 2004 4205 50  0000 L CNN
+F 0 "R2" V 2004 4205 50  0000 L CNN
 F 1 "42.2" V 2095 4205 50  0000 L CNN
 F 2 "RC1206FR-0742R2L:RESC3116X65N" H 2050 4100 50  0001 L BNN
@@
 	3300 2850 3300 3050
 $Comp
-L RMCF1206JT220R:RMCF1206JT220R R11
+L RMCF1206JT220R:RMCF1206JT220R R6
 U 1 1 61665485
 P 7500 2000
-F 0 "R11" H 7500 2242 50  0000 C CNN
+F 0 "R6" H 7500 2242 50  0000 C CNN
 F 1 "220" H 7500 2151 50  0000 C CNN
 F 2 "RMCF1206JT220R:RESC3216X70N" H 7500 2000 50  0001 L BNN
@@
 	7900 2000 8100 2000
 $Comp
-L WL-TMRC:WL-TMRC D3
+L WL-TMRC:WL-TMRC D2
 U 1 1 6161A01D
 P 7100 3450
-F 0 "D3" V 7168 3311 50  0000 R CNN
+F 0 "D2" V 7168 3311 50  0000 R CNN
 F 1 "Red" V 7077 3311 50  0000 R CNN
 F 2 "WL-TMRC:LED-5MM-ROUND" H 7100 3450 50  0001 C CNN
@@
 $EndComp
 $Comp
-L 2021-10-29_06-40-06:RNCP1206FTD100R R10
+L 2021-10-29_06-40-06:RNCP1206FTD100R R5
 U 1 1 617F85FE
 P 7450 3650
-F 0 "R10" V 7647 3729 60  0000 L CNN
+F 0 "R5" V 7647 3729 60  0000 L CNN
 F 1 "100" V 7753 3729 60  0000 L CNN
 F 2 "footprints:RNCP1206FTD100R" H 7700 3315 60  0001 C CNN
@@
 $EndComp
 $Comp
-L 2021-10-29_06-40-06:RNCP1206FTD100R R9
+L 2021-10-29_06-40-06:RNCP1206FTD100R R4
 U 1 1 617FA914
 P 7100 3650
-F 0 "R9" V 7297 3729 60  0000 L CNN
+F 0 "R4" V 7297 3729 60  0000 L CNN
 F 1 "100" V 7403 3729 60  0000 L CNN
 F 2 "footprints:RNCP1206FTD100R" H 7350 3315 60  0001 C CNN
@@
 $EndComp
 $Comp
-L 2021-10-29_06-40-06:RNCP1206FTD100R R8
+L 2021-10-29_06-40-06:RNCP1206FTD100R R3
 U 1 1 617FB26E
 P 3300 3750
-F 0 "R8" V 3497 3829 60  0000 L CNN
+F 0 "R3" V 3497 3829 60  0000 L CNN
 F 1 "100" V 3603 3829 60  0000 L CNN
 F 2 "footprints:RNCP1206FTD100R" H 3550 3415 60  0001 C CNN
@@
 $EndComp
 $Comp
-L WP7113GD:WP7113GD D2
+L WP7113GD:WP7113GD D1
 U 1 1 617D44BC
 P 3300 3450
-F 0 "D2" V 3396 3371 50  0000 R CNN
+F 0 "D1" V 3396 3371 50  0000 R CNN
 F 1 "Green" V 3305 3371 50  0000 R CNN
 F 2 "WP7113GD:LED_WP7113GD" H 3300 3450 50  0001 L BNN
@@
 $EndComp
 $Comp
-L WP7113GD:WP7113GD D4
+L WP7113GD:WP7113GD D3
 U 1 1 617DC6A4
 P 7450 3350
-F 0 "D4" V 7546 3271 50  0000 R CNN
+F 0 "D3" V 7546 3271 50  0000 R CNN
 F 1 "Green" V 7455 3271 50  0000 R CNN
 F 2 "WP7113GD:LED_WP7113GD" H 7450 3350 50  0001 L BNN
@@
 $EndComp
 $Comp
-L WP7113GD:WP7113GD D6
+L WP7113GD:WP7113GD D5
 U 1 1 617E4650
 P 8500 2000
-F 0 "D6" H 8550 1783 50  0000 C CNN
+F 0 "D5" H 8550 1783 50  0000 C CNN
 F 1 "Green" H 8550 1874 50  0000 C CNN
 F 2 "WP7113GD:LED_WP7113GD" H 8500 2000 50  0001 L BNN
@@
 Wire Bus Line
 	1950 2050 1950 2650
+Connection ~ 5850 2050
+Wire Wire Line
+	5850 2050 5850 1950
 $EndSCHEMATC
