File: Hardware/tool_circuit/raspberrypi_header.sch (KiCad schematic (older format))
At the start: 23 parts, among them J4 GPIO_CONNECTOR

Commit message: pcb revisions
Parts:
- removed H1, H2, H3, H4: MountingHole, lib:MountingHole_2.7mm_M2.5_uHAT_RPi, symbol Mechanical:MountingHole
- D1: value Green -> 3.3V
- D2: value Red -> Disable
- D3: value Green -> Enable
- D4: value Yellow -> Data_Transfer
- D5: value Green -> 5V
- LED1: value Blue -> Tool_In_Use
- TP3: value S2751-46R -> Tool_In_Use
- TP4: value S2751-46R -> 3.3V
- TP5: value S2751-46R -> GPIO1
- TP6: value S2751-46R -> Disable
- TP7: value S2751-46R -> Enable_LED
- TP8: value S2751-46R -> Data_Transfer
- renumbered R2 to R4, R3 to R5, R4 to R6, R5 to R7, R6 to R8, R7 to R9
Connections:
- net GPIO2 renamed GPIO2_SDA1
- net GPIO27 renamed GPIO27_GEN2
- net GPIO3 renamed GPIO3_SCL1
Changed lines of the file:
@@
 $Descr A4 11693 8268
 encoding utf-8
-Sheet 8 8
+Sheet 7 8
 Title ""
 Date ""
@@
 	5550 3950 6600 3950
 $Comp
-L Mechanical:MountingHole H1
-U 1 1 5C7C4C81
-P 8850 2500
-F 0 "H1" H 8950 2546 50  0000 L CNN
-F 1 "MountingHole" H 8950 2455 50  0000 L CNN
-F 2 "lib:MountingHole_2.7mm_M2.5_uHAT_RPi" H 8850 2500 50  0001 C CNN
-F 3 "~" H 8850 2500 50  0001 C CNN
-	1    8850 2500
-	1    0    0    -1
-$EndComp
-$Comp
-L Mechanical:MountingHole H2
-U 1 1 5C7C7FBC
-P 8850 2700
-F 0 "H2" H 8950 2746 50  0000 L CNN
-F 1 "MountingHole" H 8950 2655 50  0000 L CNN
-F 2 "lib:MountingHole_2.7mm_M2.5_uHAT_RPi" H 8850 2700 50  0001 C CNN
-F 3 "~" H 8850 2700 50  0001 C CNN
-	1    8850 2700
-	1    0    0    -1
-$EndComp
-$Comp
-L Mechanical:MountingHole H3
-U 1 1 5C7C8014
-P 8850 2900
-F 0 "H3" H 8950 2946 50  0000 L CNN
-F 1 "MountingHole" H 8950 2855 50  0000 L CNN
-F 2 "lib:MountingHole_2.7mm_M2.5_uHAT_RPi" H 8850 2900 50  0001 C CNN
-F 3 "~" H 8850 2900 50  0001 C CNN
-	1    8850 2900
-	1    0    0    -1
-$EndComp
-$Comp
-L Mechanical:MountingHole H4
-U 1 1 5C7C8030
-P 8850 3100
-F 0 "H4" H 8950 3146 50  0000 L CNN
-F 1 "MountingHole" H 8950 3055 50  0000 L CNN
-F 2 "lib:MountingHole_2.7mm_M2.5_uHAT_RPi" H 8850 3100 50  0001 C CNN
-F 3 "~" H 8850 3100 50  0001 C CNN
-	1    8850 3100
-	1    0    0    -1
-$EndComp
-Wire Wire Line
-	2050 2150 5050 2150
-Text Label 3250 2150 0    50   ~ 0
-GPIO2
-Text Label 3250 2250 0    50   ~ 0
-GPIO3
-$Comp
 L WP7113YD:WP7113YD D4
 U 1 1 61534E0C
 P 8100 3200
 F 0 "D4" V 8196 3121 50  0000 R CNN
-F 1 "Yellow" V 8105 3121 50  0000 R CNN
+F 1 "Data_Transfer" V 8105 3121 50  0000 R CNN
 F 2 "WP7113YD:LED_WP7113YD" H 8100 3200 50  0001 L BNN
 F 3 "" H 8100 3200 50  0001 L BNN
@@
 Text Label 2850 2750 0    50   ~ 0
 Tool_In_Use
-Text Label 4100 2150 0    50   ~ 0
-GPIO2_SDA1
 Text Label 4100 2250 0    50   ~ 0
 GPIO3_SCL1
@@
 AR Path="/61514F71/61630B5E" Ref="LED1"  Part="1"
 F 0 "LED1" V 2197 3528 60  0000 L CNN
-F 1 "Blue" V 2303 3528 60  0000 L CNN
+F 1 "Tool_In_Use" V 2303 3528 60  0000 L CNN
 F 2 "Blue LED:151034BS03000" H 2250 2940 60  0001 C CNN
 F 3 "" H 2050 3300 60  0000 C CNN
@@
 P 4950 1950
 F 0 "TP5" H 5035 2017 50  0000 L CNN
-F 1 "S2751-46R" H 5035 1926 50  0000 L CNN
+F 1 "GPIO1" H 5000 2200 50  0000 L CNN
 F 2 "S2751-46R:HARWIN_S2751-46R" H 4950 1950 50  0001 L BNN
 F 3 "" H 4950 1950 50  0001 L BNN
@@
 P 7450 2650
 F 0 "TP8" H 7535 2717 50  0000 L CNN
-F 1 "S2751-46R" H 7535 2626 50  0000 L CNN
+F 1 "Data_Transfer" H 7535 2626 50  0000 L CNN
 F 2 "S2751-46R:HARWIN_S2751-46R" H 7450 2650 50  0001 L BNN
 F 3 "" H 7450 2650 50  0001 L BNN
@@
 P 7300 2950
 F 0 "TP7" H 7215 2924 50  0000 R CNN
-F 1 "S2751-46R" H 7215 3015 50  0000 R CNN
+F 1 "Enable_LED" H 7215 3015 50  0000 R CNN
 F 2 "S2751-46R:HARWIN_S2751-46R" H 7300 2950 50  0001 L BNN
 F 3 "" H 7300 2950 50  0001 L BNN
@@
 P 6900 3150
 F 0 "TP6" H 6815 3124 50  0000 R CNN
-F 1 "S2751-46R" H 6815 3215 50  0000 R CNN
+F 1 "Disable" H 7100 3400 50  0000 R CNN
 F 2 "S2751-46R:HARWIN_S2751-46R" H 6900 3150 50  0001 L BNN
 F 3 "" H 6900 3150 50  0001 L BNN
@@
 P 3600 2950
 F 0 "TP4" H 3515 2924 50  0000 R CNN
-F 1 "S2751-46R" H 3515 3015 50  0000 R CNN
+F 1 "3.3V" H 3515 3015 50  0000 R CNN
 F 2 "S2751-46R:HARWIN_S2751-46R" H 3600 2950 50  0001 L BNN
 F 3 "" H 3600 2950 50  0001 L BNN
@@
 P 2350 2850
 F 0 "TP3" H 2265 2824 50  0000 R CNN
-F 1 "S2751-46R" H 2265 2915 50  0000 R CNN
+F 1 "Tool_In_Use" H 2265 2915 50  0000 R CNN
 F 2 "S2751-46R:HARWIN_S2751-46R" H 2350 2850 50  0001 L BNN
 F 3 "" H 2350 2850 50  0001 L BNN
@@
 	-1   0    0    1
 $EndComp
-Wire Wire Line
-	2350 2750 5050 2750
-$Comp
-L AC1206FR-07130RL:AC1206FR-07130RL R7
+$Comp
+L AC1206FR-07130RL:AC1206FR-07130RL R9
 U 1 1 61659CB7
 P 8100 3900
-F 0 "R7" V 8054 4005 50  0000 L CNN
+F 0 "R9" V 8054 4005 50  0000 L CNN
 F 1 "130" V 8145 4005 50  0000 L CNN
 F 2 "AC1206FR-07130RL:RESC3116X65N" H 8100 3900 50  0001 L BNN
@@
 $EndComp
 $Comp
-L RC1206FR-0742R2L:RC1206FR-0742R2L R2
+L RC1206FR-0742R2L:RC1206FR-0742R2L R4
 U 1 1 6165D04D
 P 2050 4100
-F 0 "R2" V 2004 4205 50  0000 L CNN
+F 0 "R4" V 2004 4205 50  0000 L CNN
 F 1 "42.2" V 2095 4205 50  0000 L CNN
 F 2 "RC1206FR-0742R2L:RESC3116X65N" H 2050 4100 50  0001 L BNN
@@
 	3300 2850 3300 3050
 $Comp
-L RMCF1206JT220R:RMCF1206JT220R R6
+L RMCF1206JT220R:RMCF1206JT220R R8
 U 1 1 61665485
 P 7500 2000
-F 0 "R6" H 7500 2242 50  0000 C CNN
+F 0 "R8" H 7500 2242 50  0000 C CNN
 F 1 "220" H 7500 2151 50  0000 C CNN
 F 2 "RMCF1206JT220R:RESC3216X70N" H 7500 2000 50  0001 L BNN
@@
 	1    0    0    -1
 $EndComp
-Connection ~ 2350 2750
 Connection ~ 5850 2150
 Wire Wire Line
@@
 Wire Wire Line
 	5550 2150 5850 2150
-Text Label 3300 2650 0    50   ~ 0
-GPIO27
-Entry Wire Line
-	1950 2650 2050 2750
-Text HLabel 1250 2050 0    50   BiDi ~ 0
-PI_CONN
-Entry Wire Line
-	1950 2550 2050 2650
-Entry Wire Line
-	1950 2250 2050 2350
-Entry Wire Line
-	1950 2050 2050 2150
-Wire Bus Line
-	1250 2050 1950 2050
-Wire Wire Line
-	5050 2250 2200 2250
-Wire Wire Line
-	2200 2250 2200 2350
-Wire Wire Line
-	2200 2350 2050 2350
-Wire Wire Line
-	2050 2650 5050 2650
 Wire Wire Line
 	5050 2550 4050 2550
@@
 P 7100 3450
 F 0 "D2" V 7168 3311 50  0000 R CNN
-F 1 "Red" V 7077 3311 50  0000 R CNN
+F 1 "Disable" V 7077 3311 50  0000 R CNN
 F 2 "WL-TMRC:LED-5MM-ROUND" H 7100 3450 50  0001 C CNN
 F 3 "" H 7100 3450 50  0001 L BNN
@@
 $EndComp
 $Comp
-L 2021-10-29_06-40-06:RNCP1206FTD100R R5
+L 2021-10-29_06-40-06:RNCP1206FTD100R R7
 U 1 1 617F85FE
 P 7450 3650
-F 0 "R5" V 7647 3729 60  0000 L CNN
+F 0 "R7" V 7647 3729 60  0000 L CNN
 F 1 "100" V 7753 3729 60  0000 L CNN
 F 2 "footprints:RNCP1206FTD100R" H 7700 3315 60  0001 C CNN
@@
 $EndComp
 $Comp
-L 2021-10-29_06-40-06:RNCP1206FTD100R R4
+L 2021-10-29_06-40-06:RNCP1206FTD100R R6
 U 1 1 617FA914
 P 7100 3650
-F 0 "R4" V 7297 3729 60  0000 L CNN
+F 0 "R6" V 7297 3729 60  0000 L CNN
 F 1 "100" V 7403 3729 60  0000 L CNN
 F 2 "footprints:RNCP1206FTD100R" H 7350 3315 60  0001 C CNN
@@
 $EndComp
 $Comp
-L 2021-10-29_06-40-06:RNCP1206FTD100R R3
+L 2021-10-29_06-40-06:RNCP1206FTD100R R5
 U 1 1 617FB26E
 P 3300 3750
-F 0 "R3" V 3497 3829 60  0000 L CNN
+F 0 "R5" V 3497 3829 60  0000 L CNN
 F 1 "100" V 3603 3829 60  0000 L CNN
 F 2 "footprints:RNCP1206FTD100R" H 3550 3415 60  0001 C CNN
@@
 P 3300 3450
 F 0 "D1" V 3396 3371 50  0000 R CNN
-F 1 "Green" V 3305 3371 50  0000 R CNN
+F 1 "3.3V" V 3305 3371 50  0000 R CNN
 F 2 "WP7113GD:LED_WP7113GD" H 3300 3450 50  0001 L BNN
 F 3 "" H 3300 3450 50  0001 L BNN
@@
 P 7450 3350
 F 0 "D3" V 7546 3271 50  0000 R CNN
-F 1 "Green" V 7455 3271 50  0000 R CNN
+F 1 "Enable" V 7455 3271 50  0000 R CNN
 F 2 "WP7113GD:LED_WP7113GD" H 7450 3350 50  0001 L BNN
 F 3 "" H 7450 3350 50  0001 L BNN
@@
 P 8500 2000
 F 0 "D5" H 8550 1783 50  0000 C CNN
-F 1 "Green" H 8550 1874 50  0000 C CNN
+F 1 "5V" H 8550 1874 50  0000 C CNN
 F 2 "WP7113GD:LED_WP7113GD" H 8500 2000 50  0001 L BNN
 F 3 "" H 8500 2000 50  0001 L BNN
@@
 Wire Wire Line
 	5850 2050 5850 1950
-Wire Bus Line
-	1950 2050 1950 2650
+Text GLabel 2600 2150 0    50   BiDi ~ 0
+GPIO2_SDA1
+Wire Wire Line
+	5050 2150 2600 2150
+Text GLabel 2700 2250 0    50   BiDi ~ 0
+GPIO3_SCL1
+Connection ~ 2350 2750
+Wire Wire Line
+	2350 2750 5050 2750
+Wire Wire Line
+	5050 2250 2700 2250
+Text GLabel 2750 2650 0    50   BiDi ~ 0
+GPIO27_GEN2
+Text GLabel 2050 2750 0    50   BiDi ~ 0
+GPIO22_GEN3
+Wire Wire Line
+	5050 2650 2750 2650
 $EndSCHEMATC
