File: Hardware/tool_circuit/raspberrypi_header.sch (KiCad schematic (older format))
At the start: 20 parts, among them J4 GPIO_CONNECTOR

Commit message: pulling
Connections:
- net GPIO22_GEN3: no longer LED1.2, R1.1, TP3.1
- new net Time_of_use: LED1.2, R1.1, TP3.1
Changed lines of the file:
@@
 Wire Wire Line
 	7000 2000 7100 2000
-Text Label 3600 2750 0    50   ~ 0
-Tool_In_Use
 Text Label 4100 2250 0    50   ~ 0
 GPIO3_SCL1
@@
 P 7450 2650
 F 0 "TP8" H 7535 2717 50  0000 L CNN
-F 1 "Data_Transfer" H 7535 2626 50  0000 L CNN
+F 1 "Data_Transfer" H 7250 2900 50  0000 L CNN
 F 2 "S2751-46R:HARWIN_S2751-46R" H 7450 2650 50  0001 L BNN
 F 3 "" H 7450 2650 50  0001 L BNN
@@
 GPIO27_GEN2
 Text GLabel 2050 2750 0    50   BiDi ~ 0
-GPIO22_GEN3
+Time_of_use
 Wire Wire Line
 	5050 2650 2750 2650
