File: Hardware/tool_circuit/tool_circuit.kicad_pcb (KiCad board)
At the start: 2 copper layers, 12 parts, among them J1 Conn_01x03_Female, U1 DHT11, U2 TPS563211DRLR

Commit message: pcb layout and schematic changes
Parts:
- removed R1: RNCP1206FTD4K99, RNCP1206FTD4K99:RNCP1206FTD4K99
- removed U1: DHT11, Sensor:Aosong_DHT11_5.5x12.0_P2.54mm
- added J2: Conn_01x08_Female, Connector_PinHeader_2.54mm:PinHeader_1x08_P2.54mm_Vertical, F.Cu at (158.2, 89.4)
- added J3: Conn_01x03_Female, Connector_PinHeader_2.54mm:PinHeader_1x03_P2.54mm_Vertical, F.Cu at (164.3, 89.3)
- moved J1 82.5 mm to (164.4, 102.1)
- moved C2 75.9 mm to (149.5, 90.9)
- moved L1 74.3 mm to (146.7, 101.9)
- moved C1 73.2 mm to (143.3, 90.2)
- moved U2 73.1 mm to (140.9, 85.1)
- moved R2 65.7 mm to (144.8, 85.1)
- moved C4 64.3 mm to (150.3, 93.1)
- moved C3 63.3 mm to (150.4, 88.6)
- moved R4 61.4 mm to (149.0, 86.2)
- moved R3 54.2 mm to (149.4, 84.7)
Connections:
- net Net-(J1-Pad2) renamed /Vibration_Sensor/GPIO_27
- J1 pad 1: Net-(J1-Pad1) -> +5V
- J1 pad 3: Net-(J1-Pad3) -> GND

Commit message: schematic updates
Parts:
- removed the J2 at (158.2, 89.4)
- added H1: MountingHole, lib:MountingHole_2.7mm_M2.5_uHAT_RPi, F.Cu at (157.9, 87.6)
- added H2: MountingHole, lib:MountingHole_2.7mm_M2.5_uHAT_RPi, F.Cu at (215.9, 87.6)
- added H3: MountingHole, lib:MountingHole_2.7mm_M2.5_uHAT_RPi, F.Cu at (215.9, 110.6)
- added H4: MountingHole, lib:MountingHole_2.7mm_M2.5_uHAT_RPi, F.Cu at (157.9, 110.6)
- added J3: Conn_01x08_Female, Connector_PinHeader_2.54mm:PinHeader_1x08_P2.54mm_Vertical, F.Cu at (94.6, 84.6)
- added R10: 100, RESC3115X60N, F.Cu at (82.2, 97.3)
- added R12: 100, RESC3115X60N, F.Cu at (82.2, 100.6)
- added R14: 100, RESC3115X60N, F.Cu at (87.8, 97.3)
- C1: value KCM55QR7YA226KH01L -> 22UF
- C2: value CGA3E2X7R1H104K080AA -> 0.1UF; footprint CGA3E2X7R1H104K080AA:CAPC1608X90N -> CAPC3216X180N
- C3: value CL31B104KBCNNNC -> 0.1UF
- C4: value 12063D106MAT2A -> 10UF
- J1: value Conn_01x03_Female -> EJ503A; footprint Connector_PinHeader_2.54mm:PinHeader_1x03_P2.54mm_Vertical -> lib:PinSocket_2x20_P2.54mm_Vertical_Centered_Anchor; moved to B.Cu
- L1: value SDR1307-4R7ML -> 4.7UH
- R1: renamed from R2; value RNCP1206FTD10K0 -> 10K
- R2: renamed from R3; value RC0603FR-0782KL -> 82K
- R3: renamed from R4; value CRCW040210K0DHEDP -> 10K
- moved C3 77.0 mm to (73.5, 84.4)
- moved C4 77.0 mm to (73.4, 88.8)
- moved R3 77.0 mm to (72.1, 82.0)
- moved L1 77.0 mm to (69.8, 97.6)
- moved R2 77.0 mm to (72.5, 80.5)
- moved U1 77.0 mm to (64.0, 80.8)
- moved C1 77.0 mm to (66.4, 85.9)
- moved J2 77.0 mm to (87.4, 85.0)
- moved R1 77.0 mm to (67.9, 80.8)
- moved C2 69.6 mm to (79.9, 88.5)
- moved J1 13.3 mm to (162.7, 88.9), turned to 270 degrees
- renumbered J3 to J2, U2 to U1
Connections:
- net /Temp_Sense/GPIO_17 renamed /Temp_Sense/GPIO27
- C1 pad 2: /Power_Src/5V Regulator/12V_BATTERY -> +12V
- C2 pad 2: /Power_Src/5V Regulator/12V_BATTERY -> +12V
- C4 pad 2: /Power_Src/5V Regulator/5V -> +5V
- J1 pad 1: +5V -> +12V
- J1 pad 2: /Vibration_Sensor/GPIO_27 -> GND
- J2 pad 1: +5V -> +3V3
- L1 pad 1: /Power_Src/5V Regulator/5V -> +5V
- R1 pad 2: /Power_Src/5V Regulator/5V -> +5V
- R2 pad 2: /Power_Src/5V Regulator/5V -> +5V
- U1 pad 2: /Power_Src/5V Regulator/12V_BATTERY -> +12V
Routing:
- added copper zone on B.Cu, net GND
- added copper zone on F.Cu, net GND
Other:
- board outline added: 65 x 30 mm
- net class Default: clearance 0.254 -> 0.2; trace_width 0.254 -> 0.25; via_dia 0.7 -> 0.8
- rule pad_to_mask_clearance: 0.0508 -> 0.051
- rule trace_clearance: 0.254 -> 0.2
- rule trace_min: 0.1524 -> 0.2
- rule via_min_drill: 0.254 -> 0.3
- rule via_min_size: 0.508 -> 0.4
- board text added: "Board Corner Radius = 3mm All holes are M2.5"
- board text added: "Board dimensions are on Cmts (Comments) layer. Deselect it in Layers Manager to make them invisible. GPIO connector nets are not connected, these will get updated as per your schematic/netlist."

Commit message: PCB changes
Parts:
- removed R14: 100, RESC3115X60N
- added D1: Green, WP7113GD:LED_WP7113GD, F.Cu at (119.6, 56.7)
- added D2: Green, WP7113GD:LED_WP7113GD, F.Cu at (126.8, -3.37)
- added D3: Red, WL-TMRC:LED-5MM-ROUND, F.Cu at (197.8, 164.3)
- added D4: Green, WP7113GD:LED_WP7113GD, F.Cu at (135.1, -3.37)
- added D5: Yellow, WP7113YD:LED_WP7113YD, F.Cu at (198.2, 156.3)
- added D6: Green, WP7113GD:LED_WP7113GD, F.Cu at (143.4, -3.37)
- added J4: GPIO_CONNECTOR, lib:PinSocket_2x20_P2.54mm_Vertical_Centered_Anchor, F.Cu at (119.0, 18.9)
- added LED1: Blue, Blue LED:151034BS03000, F.Cu at (205.3, 159.9)
- added R11: 220, RMCF1206JT220R:RESC3216X70N, F.Cu at (87.8, 97.3)
- added R4: 82K, ul_RC0603FR-0782KL:RC0603FR-0782KL, F.Cu at (163.8, 178.5)
- added R5: 10K, CRCW040210K0DHEDP:RESC1005X40N, F.Cu at (167.2, 178.3)
- added R6: 10k, RNCP1206FTD10K0:RESC3115X60N, F.Cu at (170.1, 153.8)
- added R7: 42.2, RC1206FR-0742R2L:RESC3116X65N, F.Cu at (212.0, 158.8)
- added R8: 100, footprints:RNCP1206FTD100R, F.Cu at (82.2, 97.3)
- added R9: 100, footprints:RNCP1206FTD100R, F.Cu at (219.3, 153.8)
- added S1: 1825255-1, 1825255-1:SW_1825255-1, F.Cu at (162.4, 161.5)
- added TP1: S2751-46R, S2751-46R:HARWIN_S2751-46R, F.Cu at (160.0, 178.9)
- added TP2: S2751-46R, S2751-46R:HARWIN_S2751-46R, F.Cu at (165.6, 175.6)
- added TP3: S2751-46R, S2751-46R:HARWIN_S2751-46R, F.Cu at (211.8, 162.0)
- added TP4: S2751-46R, S2751-46R:HARWIN_S2751-46R, F.Cu at (217.3, 158.7)
- added TP5: S2751-46R, S2751-46R:HARWIN_S2751-46R, F.Cu at (216.3, 162.0)
- added TP6: S2751-46R, S2751-46R:HARWIN_S2751-46R, F.Cu at (209.7, 165.0)
- added TP7: S2751-46R, S2751-46R:HARWIN_S2751-46R, F.Cu at (209.5, 168.1)
- added TP8: S2751-46R, S2751-46R:HARWIN_S2751-46R, F.Cu at (221.8, 157.0)
- J1: footprint lib:PinSocket_2x20_P2.54mm_Vertical_Centered_Anchor -> EJ503A:MPD_EJ503A
- R1: value 10K -> 820; footprint RNCP1206FTD10K0:RESC3115X60N -> CRGCQ1206F820R:RESC3115X65N
- R10: footprint RESC3115X60N -> footprints:RNCP1206FTD100R
- R12: value 100 -> 130; footprint RESC3115X60N -> AC1206FR-07130RL:RESC3116X65N
- R2: value 82K -> 0; footprint ul_RC0603FR-0782KL:RC0603FR-0782KL -> RK73Z2BTTD:RK73Z2BTTD
- R3: footprint CRCW040210K0DHEDP:RESC1005X40N -> RNCP1206FTD10K0:RESC3115X60N
- moved R10 140.8 mm to (204.3, 167.5)
- moved R12 137.8 mm to (204.4, 164.2)
- moved R3 128.6 mm to (160.2, 175.7)
- moved R1 4.66 mm to (72.5, 80.5)
- moved R2 1.57 mm to (72.1, 82.0)
Connections:
- R1 pad 1: Net-(R1-Pad1) -> Net-(D1-PadC)
- R1 pad 2: +5V -> GND
- R2 pad 2: +5V -> GND
- R3 pad 1: Net-(R2-Pad1) -> Net-(R3-Pad1)
- R3 pad 2: GND -> +5V
- U1 pad 1: Net-(R1-Pad1) -> Net-(R3-Pad1)
- U1 pad 6: Net-(R6-Pad1) -> Net-(R2-Pad1)
- U1 pad 8: Net-(R2-Pad1) -> Net-(R4-Pad1)

Commit message: layout
Parts:
- removed C3: 0.1UF, CL31B104KBCNNNC:CAPC3216X180N
- removed C4: 10UF, 12063D106MAT2A:CAPC3216X178N
- removed D6: Green, WP7113GD:LED_WP7113GD
- removed R10, R8, R9: 100, footprints:RNCP1206FTD100R
- removed R11: 220, RMCF1206JT220R:RESC3216X70N
- removed R12: 130, AC1206FR-07130RL:RESC3116X65N
- added CR1: B380-13-F, B380-13-F:B380-13-F, F.Cu at (165.7, 109.0)
- C1: value 22UF -> 100uF; footprint KCM55QR7YA226KH01L:CAPC6153X390N -> EEUFS1K101:CAPPRD500W60D1000H1250
- C2: value 0.1UF -> 1000uF; footprint CAPC3216X180N -> URS1E102MHD1TO:URS1E102MHD1TO
- D2: value Green -> Red; footprint WP7113GD:LED_WP7113GD -> WL-TMRC:LED-5MM-ROUND
- D3: value Red -> Green; footprint WL-TMRC:LED-5MM-ROUND -> WP7113GD:LED_WP7113GD
- D4: value Green -> Yellow; footprint WP7113GD:LED_WP7113GD -> WP7113YD:LED_WP7113YD
- D5: value Yellow -> Green; footprint WP7113YD:LED_WP7113YD -> WP7113GD:LED_WP7113GD
- J1: moved to F.Cu
- J4: moved to B.Cu
- L1: value 4.7UH -> 100 uH; footprint ul_SDR1307-4R7ML:SDR1307-4R7ML -> IHLP-4040DZ_VIS:IHLP4040DZER101M11
- R1: value 820 -> 10k; footprint CRGCQ1206F820R:RESC3115X65N -> RNCP1206FTD10K0:RESC3115X60N
- R2: value 0 -> 42.2; footprint RK73Z2BTTD:RK73Z2BTTD -> RC1206FR-0742R2L:RESC3116X65N
- R3: value 10K -> 100; footprint RNCP1206FTD10K0:RESC3115X60N -> footprints:RNCP1206FTD100R
- R4: value 82K -> 100; footprint ul_RC0603FR-0782KL:RC0603FR-0782KL -> footprints:RNCP1206FTD100R
- R5: value 10K -> 100; footprint CRCW040210K0DHEDP:RESC1005X40N -> footprints:RNCP1206FTD100R
- R6: value 10k -> 220; footprint RNCP1206FTD10K0:RESC3115X60N -> RMCF1206JT220R:RESC3216X70N
- R7: value 42.2 -> 130; footprint RC1206FR-0742R2L:RESC3116X65N -> AC1206FR-07130RL:RESC3116X65N
- U1: value TPS563211DRLR -> LM2576D2TR4-5G; footprint ul_TPS563211DRLR:TPS563211DRLR -> LM2576D2TR4-5G:D2PAK-5
- moved C1 142.0 mm to (206.6, 108.3)
- moved D4 138.8 mm to (185.8, 125.8)
- moved C2 135.4 mm to (215.0, 97.4), turned to 180 degrees
- moved L1 123.1 mm to (192.9, 96.3), turned to 180 degrees
- moved D2 121.8 mm to (143.3, 117.3)
- moved U1 113.7 mm to (176.7, 96.3)
- moved J2 111.8 mm to (196.0, 111.8), turned to 180 degrees
- moved R2 105.6 mm to (174.4, 108.5), turned to 90 degrees
- moved R1 103.2 mm to (171.8, 108.5), turned to 90 degrees
- moved J4 96.5 mm to (186.9, 87.6), turned to 270 degrees
- moved D1 88.3 mm to (152.4, 138.7)
- moved J3 81.8 mm to (174.1, 103.5), turned to 270 degrees
- moved D3 73.3 mm to (230.0, 98.4)
- moved S1 57.1 mm to (185.0, 109.0), turned to 270 degrees
- moved D5 56.8 mm to (228.5, 108.3)
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Connections:
- C2 pad 1: GND -> +5V
- C2 pad 2: +12V -> GND
- D1 pad A: +12V -> +3V3
- D4 pad A: /raspberrypi_header.sch/Enable_LED -> /raspberrypi_header.sch/Data_Transfer
- D5 pad A: /raspberrypi_header.sch/Data_Transfer -> Net-(D5-PadA)
- D5 pad C: Net-(D5-PadC) -> GND
- L1 pad 2: Net-(C3-Pad1) -> Net-(CR1-Pad1)
- R1 pad 1: Net-(D1-PadC) -> Net-(R1-Pad1)
- R2 pad 1: Net-(R2-Pad1) -> Net-(LED1-Pad1)
- R3 pad 1: Net-(R3-Pad1) -> Net-(D1-PadC)
- R3 pad 2: +5V -> GND
- R4 pad 1: Net-(R4-Pad1) -> Net-(D2-Pad1)
- R4 pad 2: +5V -> GND
- R5 pad 1: Net-(R4-Pad1) -> Net-(D3-PadC)
- R6 pad 1: Net-(R6-Pad1) -> +5V
- R6 pad 2: GND -> Net-(D5-PadA)
- R7 pad 1: Net-(LED1-Pad1) -> Net-(D4-PadC)
- S1 pad 3: Net-(R6-Pad1) -> Net-(R1-Pad1)
- U1 pad 1: Net-(R3-Pad1) -> +12V
- U1 pad 2: +12V -> Net-(CR1-Pad1)
- U1 pad 3: Net-(C3-Pad1) -> GND
- U1 pad 4: GND -> +5V
- U1 pad 5: Net-(C3-Pad2) -> GND
- U1 pad 6: Net-(R2-Pad1) -> GND
Other:
- net class Default: clearance 0.2 -> 0.1524; trace_width 0.25 -> 0.1524; via_dia 0.8 -> 0.6858; via_drill 0.4 -> 0.3302
- rule pad_to_mask_clearance: 0.051 -> 0.0508
- rule trace_clearance: 0.2 -> 0.1524
- rule trace_min: 0.2 -> 0.1524
- rule via_min_drill: 0.3 -> 0.254
- rule via_min_size: 0.4 -> 0.508

Commit message: layout
Parts:
- removed H1, H2, H3, H4: MountingHole, lib:MountingHole_2.7mm_M2.5_uHAT_RPi
- removed S1: 1825255-1, 1825255-1:SW_1825255-1
- added SW1: 1825255-1, ul_1825255-1:1825255-1, F.Cu at (136.0, 98.6)
- moved TP4 116.0 mm to (121.6, 56.5), turned to 90 degrees
- moved TP5 116.0 mm to (108.3, 59.2), turned to 90 degrees
- moved D5 111.8 mm to (119.1, 85.2)
- moved C2 109.7 mm to (105.3, 97.4), turned to 0 degrees
- moved TP3 106.9 mm to (111.1, 83.2), turned to 90 degrees
- moved LED1 106.0 mm to (107.8, 77.3)
- moved TP8 104.6 mm to (123.8, 60.2), turned to 180 degrees
- moved TP7 93.3 mm to (160.9, 57.4), turned to 180 degrees
- moved TP2 90.9 mm to (104.8, 88.8), turned to 180 degrees
- moved R7 90.3 mm to (124.3, 90.8), turned to 180 degrees
- moved C1 87.3 mm to (120.0, 97.6), turned to 180 degrees
- moved J3 85.0 mm to (103.7, 55.9), turned to 0 degrees
- moved TP6 82.5 mm to (144.3, 79.5)
- moved R2 74.6 mm to (104.6, 82.2), turned to 0 degrees
- moved D3 72.1 mm to (160.1, 80.5)
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Routing:
- net /raspberrypi_header.sch/Data_Transfer: track 0.00 -> 241.6 mm
- net Net-(CR1-Pad1): track 0.00 -> 163.3 mm
- net +3V3: track 0.00 -> 156.1 mm
- net /raspberrypi_header.sch/Disable_LED: track 0.00 -> 144.2 mm
- net +5V: track 0.00 -> 136.0 mm
- net /raspberrypi_header.sch/Enable_LED: track 0.00 -> 127.9 mm
- net +12V: track 0.00 -> 70.7 mm
- net /raspberrypi_header.sch/GPIO22_GEN3: track 0.00 -> 37.1 mm
- net Net-(D5-PadA): track 0.00 -> 8.52 mm
- net Net-(R1-Pad1): track 0.00 -> 8.51 mm
- net Net-(D1-PadC): track 0.00 -> 7.95 mm
- net Net-(D2-Pad1): track 0.00 -> 7.89 mm
- net Net-(LED1-Pad1): track 0.00 -> 6.82 mm
- net Net-(D4-PadC): track 0.00 -> 5.68 mm
- net Net-(D3-PadC): track 0.00 -> 4.86 mm
Other:
- board size 65 x 30 mm -> 65 x 56.7 mm

Commit message: pcb revisions
Parts:
- removed R1: 10k, RNCP1206FTD10K0:RESC3115X60N
- added D6: 12V, WP7113GD:LED_WP7113GD, F.Cu at (109.6, 79.7)
- added R8: 220, RMCF1206JT220R:RESC3216X70N, F.Cu at (147.4, 71.3)
- added R9: 130, AC1206FR-07130RL:RESC3116X65N, F.Cu at (148.8, 87.2)
- D1: value Green -> 3.3V
- D2: value Red -> Disable
- D3: value Green -> Enable
- D4: value Yellow -> Data_Transfer
- D5: value Green -> 5V
- J2: value Conn_01x03_Female -> Temp_Sense
- J3: value Conn_01x08_Female -> Accel.
- LED1: value Blue -> Tool_In_Use
- R2: value 42.2 -> 820; footprint RC1206FR-0742R2L:RESC3116X65N -> CRGCQ1206F820R:RESC3115X65N
- R3: value 100 -> 10k; footprint footprints:RNCP1206FTD100R -> RNCP1206FTD10K0:RESC3115X60N
- R4: value 100 -> 42.2; footprint footprints:RNCP1206FTD100R -> RC1206FR-0742R2L:RESC3116X65N
- R6: value 220 -> 100; footprint RMCF1206JT220R:RESC3216X70N -> footprints:RNCP1206FTD100R
- R7: value 130 -> 100; footprint AC1206FR-07130RL:RESC3116X65N -> footprints:RNCP1206FTD100R
- SW1: value 1825255-1 -> Switch
- TP1: value S2751-46R -> Vin
- TP2: value S2751-46R -> 5V_Reg_Vout
- TP3: value S2751-46R -> Tool_In_Use
- TP4: value S2751-46R -> 3.3V
- TP5: value S2751-46R -> GPIO1
- TP6: value S2751-46R -> Disable
- TP7: value S2751-46R -> Enable_LED
- TP8: value S2751-46R -> Data_Transfer
- moved TP1 58.3 mm to (103.3, 48.5)
- moved J3 57.1 mm to (160.8, 56.7)
- moved LED1 48.9 mm to (152.7, 58.0)
- moved TP8 40.9 mm to (159.2, 80.6)
- moved TP3 40.5 mm to (146.3, 63.1), turned to 180 degrees
- moved U1 39.2 mm to (106.7, 66.0)
- moved D5 38.8 mm to (154.2, 68.7)
- moved R5 34.1 mm to (120.7, 88.1)
- moved R4 33.5 mm to (146.6, 58.6), turned to 90 degrees
- moved TP4 31.9 mm to (126.9, 88.0), turned to 0 degrees
- moved TP7 25.5 mm to (140.3, 72.4)
- moved D4 24.1 mm to (151.3, 80.1), turned to 0 degrees
- moved TP2 20.2 mm to (117.0, 72.6)
- moved R6 19.8 mm to (133.6, 87.4)
- moved TP6 19.1 mm to (125.9, 74.5), turned to 180 degrees
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Connections:
- J2 pad 2: /Temp_Sense/GPIO27 -> GPIO27_GEN2
- J3 pad 7: /Accelerometer.sch/GPIO2 -> GPIO2_SDA1
- J3 pad 8: /Accelerometer.sch/GPIO3 -> GPIO3_SCL1
- J4 pad 13: /raspberrypi_header.sch/GPIO27 -> GPIO27_GEN2
- J4 pad 15: /raspberrypi_header.sch/GPIO22_GEN3 -> GPIO22_GEN3
- J4 pad 3: /raspberrypi_header.sch/GPIO2 -> GPIO2_SDA1
- J4 pad 5: /raspberrypi_header.sch/GPIO3 -> GPIO3_SCL1
- LED1 pad 2: /raspberrypi_header.sch/GPIO22_GEN3 -> GPIO22_GEN3
- R2 pad 1: Net-(LED1-Pad1) -> Net-(D6-PadC)
- R3 pad 1: Net-(D1-PadC) -> Net-(R3-Pad1)
- R4 pad 1: Net-(D2-Pad1) -> Net-(LED1-Pad1)
- R5 pad 1: Net-(D3-PadC) -> Net-(D1-PadC)
- R6 pad 1: +5V -> Net-(D2-Pad1)
- R6 pad 2: Net-(D5-PadA) -> GND
- R7 pad 1: Net-(D4-PadC) -> Net-(D3-PadC)
- SW1 pad 1: +3V3 -> +5V
- SW1 pad 2: /Time_of_Use/GPIO22 -> GPIO22_GEN3
- SW1 pad 3: Net-(R1-Pad1) -> Net-(R3-Pad1)
- TP3 pad 1: /raspberrypi_header.sch/GPIO22_GEN3 -> GPIO22_GEN3
Routing:
- net /raspberrypi_header.sch/Data_Transfer: track 241.6 -> 49.3 mm
- net Net-(CR1-Pad1): track 163.3 -> 29.9 mm, vias 0 -> 2
- net GPIO22_GEN3: track 0.00 -> 110.1 mm, vias 0 -> 1
- net /raspberrypi_header.sch/Disable_LED: track 144.2 -> 42.0 mm, vias 0 -> 1
- net /raspberrypi_header.sch/Enable_LED: track 127.9 -> 35.8 mm, vias 0 -> 2
- net GPIO2_SDA1: track 0.00 -> 65.4 mm, vias 0 -> 1
- net GPIO3_SCL1: track 0.00 -> 58.3 mm
- net +3V3: track 156.1 -> 112.9 mm, vias 0 -> 2
- net +12V: track 70.7 -> 107.9 mm, vias 0 -> 1
- net /raspberrypi_header.sch/GPIO22_GEN3: track 37.1 -> 0.00 mm
- net GPIO27_GEN2: track 0.00 -> 20.9 mm
- net +5V: track 136.0 -> 148.9 mm, vias 0 -> 4
- net GND: track 0.00 -> 11.4 mm, vias 0 -> 8
- net Net-(R1-Pad1): track 8.51 -> 0.00 mm
- net Net-(R3-Pad1): track 0.00 -> 8.49 mm
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Other:
- board size 65 x 56.7 mm -> 65.2 x 62.6 mm
- net class Default: clearance 0.1524 -> 0.254; trace_width 0.1524 -> 0.254
- rule trace_clearance: 0.1524 -> 0.254
- rule trace_min: 0.1524 -> 0.254
- board text added: "Capstone PCB By: Komal Javed"

Commit message: PCB revisions
Parts:
- TP1: value Vin -> Vin_tp
- TP2: value 5V_Reg_Vout -> 5V_Reg_Vout_tp
- TP3: value Tool_In_Use -> Tool_In_Use_tp
- TP4: value 3.3V -> 3.3V_tp
- TP5: value GPIO1 -> GPIO1_tp
- TP6: value Disable -> Disable_tp
- TP7: value Enable_LED -> Enable_LED_tp
- TP8: value Data_Transfer -> Data_Transfer_tp
- moved U1 0.54 mm to (106.5, 65.5)
Routing:
- net GPIO2_SDA1: track 65.4 -> 79.1 mm, vias 1 -> 2
- net +5V: track 148.9 -> 155.7 mm
- net +12V: track 107.9 -> 101.1 mm
- net GND: track 11.4 -> 6.13 mm, vias 8 -> 5
- net +3V3: track 112.9 -> 116.8 mm
- net GPIO27_GEN2: track 20.9 -> 24.1 mm
- net GPIO22_GEN3: track 110.1 -> 112.1 mm, vias 1 -> 0
- net /raspberrypi_header.sch/Enable_LED: track 35.8 -> 34.3 mm, vias 2 -> 3
