File: Hardware/tool_circuit/tool_circuit.kicad_pcb (KiCad board)
At the start: 2 copper layers, 65.2 x 62.6 mm, 33 parts, among them J1 EJ503A, J2 Temp_Sense, J3 Accel., J4 GPIO_CONNECTOR, SW1 Switch, U1 LM2576D2TR4-5G

Commit message: gerber files
Parts:
- moved TP1 30.5 mm to (103.0, 79.0)
- moved J1 5.85 mm to (156.8, 92.1), turned to 0 degrees
Routing:
- net +12V: track 101.1 -> 75.0 mm, vias 1 -> 0
Other:
- rule via_min_size: 0.508 -> 0.6
Changed lines of the file:
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@@
     (thickness 1.6)
     (drawings 20)
-    (tracks 193)
+    (tracks 186)
     (zones 0)
     (modules 33)
@@
   )
   (layers
-    (0 F.Cu power)
+    (0 F.Cu signal)
     (31 B.Cu signal)
     (32 B.Adhes user)
@@
     (via_size 0.6858)
     (via_drill 0.3302)
-    (via_min_size 0.508)
+    (via_min_size 0.6)
     (via_min_drill 0.254)
     (uvia_size 0.6858)
     (uvia_drill 0.3302)
     (uvias_allowed no)
-    (uvia_min_size 0.508)
+    (uvia_min_size 0.6)
     (uvia_min_drill 0.254)
     (edge_width 0.15)
@@
     (pcbplotparams
       (layerselection 0x010fc_ffffffff)
-      (usegerberextensions false)
+      (usegerberextensions true)
       (usegerberattributes false)
       (usegerberadvancedattributes false)
       (creategerberjobfile false)
       (excludeedgelayer true)
-      (linewidth 0.100000)
+      (linewidth 0.153300)
       (plotframeref false)
       (viasonmask false)
@@
       (plotinvisibletext false)
       (padsonsilk false)
-      (subtractmaskfromsilk false)
+      (subtractmaskfromsilk true)
       (outputformat 1)
       (mirror false)
-      (drillshape 1)
+      (drillshape 0)
       (scaleselection 1)
-      (outputdirectory ""))
+      (outputdirectory "Capstone_gerbers/"))
   )
   (net 0 "")
@@
   )
   (module EJ503A:MPD_EJ503A (layer F.Cu)
-    (at 158.8526 97.603 180)
+    (at 156.846 92.1054)
     (fp_text reference J1 (at 0 0.762 180) (layer F.SilkS)
       (effects (font (size 1.4 1.4) (thickness 0.15)))
@@
     (fp_line (start -4.5 -2.96) (end -4.5 7.74) (layer F.Fab) (width 0.127))
     (fp_line (start -4.5 -3.45) (end -4.5 -2.96) (layer F.Fab) (width 0.127))
-    (pad 3 thru_hole oval (at 4.65 0 180) (size 1.9 3.8) (drill oval 0.76 3.05) (layers *.Cu *.Mask)
-      (net 1 GND))
-    (pad 2 thru_hole oval (at 0 3.25 180) (size 3.8 1.9) (drill oval 3.05 0.76) (layers *.Cu *.Mask)
-      (net 1 GND))
-    (pad 1 thru_hole oval (at 0 -2.68 180) (size 3.8 1.9) (drill oval 3.05 0.76) (layers *.Cu *.Mask)
+    (pad 3 thru_hole oval (at 4.65 0) (size 1.9 3.8) (drill oval 0.76 3.05) (layers *.Cu *.Mask)
+      (net 1 GND))
+    (pad 2 thru_hole oval (at 0 3.25) (size 3.8 1.9) (drill oval 3.05 0.76) (layers *.Cu *.Mask)
+      (net 1 GND))
+    (pad 1 thru_hole oval (at 0 -2.68) (size 3.8 1.9) (drill oval 3.05 0.76) (layers *.Cu *.Mask)
       (net 4 +12V))
   )
   (module S2751-46R:HARWIN_S2751-46R (layer F.Cu)
-    (at 103.2774 48.5178 180)
+    (at 103.0488 78.9978 180)
     (fp_text reference TP1 (at 0.44 -1.808) (layer F.SilkS)
       (effects (font (size 0.8 0.8) (thickness 0.15)))
@@
       (effects (font (size 0.8 0.8) (thickness 0.15)))
     )
-    (fp_text value Data_Transfer_tp (at 0.0762 -3.3274) (layer F.Fab)
+    (fp_text value Data_Transfer_tp (at -0.4318 2.2352) (layer F.Fab)
       (effects (font (size 0.8 0.8) (thickness 0.15)))
     )
@@
   (segment (start 108.1796 72.8002) (end 108.1796 70.057) (width 0.508) (layer F.Cu) (net 3))
   (segment (start 110.7958 50.4736) (end 108.2558 50.4736) (width 0.508) (layer B.Cu) (net 3))
-  (segment (start 108.2558 50.4736) (end 100.8644 57.865) (width 0.508) (layer B.Cu) (net 3))
-  (segment (start 100.8644 57.865) (end 100.8644 73.5876) (width 0.508) (layer B.Cu) (net 3))
   (segment (start 100.8644 73.5876) (end 101.8804 74.6036) (width 0.508) (layer B.Cu) (net 3))
   (segment (start 106.3762 74.6036) (end 108.1796 72.8002) (width 0.508) (layer B.Cu) (net 3))
   (segment (start 101.8804 74.6036) (end 106.3762 74.6036) (width 0.508) (layer B.Cu) (net 3))
-  (segment (start 130.351901 103.597701) (end 124.3448 97.5906) (width 0.508) (layer B.Cu) (net 4))
-  (segment (start 116.166 89.4118) (end 124.3448 97.5906) (width 0.508) (layer B.Cu) (net 4))
-  (segment (start 115.063 89.4118) (end 116.166 89.4118) (width 0.508) (layer B.Cu) (net 4))
-  (segment (start 108.5098 86.5416) (end 111.38 89.4118) (width 0.508) (layer B.Cu) (net 4))
-  (via (at 108.5098 86.5416) (size 0.6858) (drill 0.3302) (layers F.Cu B.Cu) (net 4))
-  (segment (start 155.537899 103.597701) (end 158.8526 100.283) (width 0.508) (layer B.Cu) (net 4))
-  (segment (start 130.351901 103.597701) (end 155.537899 103.597701) (width 0.508) (layer B.Cu) (net 4))
-  (segment (start 108.332 86.3638) (end 108.5098 86.5416) (width 0.508) (layer B.Cu) (net 4))
-  (segment (start 108.332 79.6582) (end 108.332 86.3638) (width 0.508) (layer B.Cu) (net 4))
-  (segment (start 111.38 89.4118) (end 115.063 89.4118) (width 0.508) (layer B.Cu) (net 4))
-  (segment (start 100.671399 67.654199) (end 103.0488 70.0316) (width 0.254) (layer F.Cu) (net 4))
-  (segment (start 100.671399 51.123801) (end 100.671399 67.654199) (width 0.254) (layer F.Cu) (net 4))
-  (segment (start 103.2774 48.5178) (end 100.671399 51.123801) (width 0.254) (layer F.Cu) (net 4))
-  (segment (start 103.0488 74.375) (end 108.332 79.6582) (width 0.254) (layer F.Cu) (net 4))
-  (segment (start 103.0488 70.0316) (end 103.0488 74.375) (width 0.254) (layer F.Cu) (net 4))
+  (segment (start 100.8644 57.865) (end 100.8644 73.5876) (width 0.508) (layer B.Cu) (net 3))
+  (segment (start 108.2558 50.4736) (end 100.8644 57.865) (width 0.508) (layer B.Cu) (net 3))
+  (segment (start 103.0488 70.0316) (end 103.0488 78.9978) (width 0.508) (layer F.Cu) (net 4))
+  (segment (start 107.6716 78.9978) (end 108.332 79.6582) (width 0.508) (layer F.Cu) (net 4))
+  (segment (start 103.0488 78.9978) (end 107.6716 78.9978) (width 0.508) (layer F.Cu) (net 4))
+  (segment (start 108.332 81.5778) (end 124.3448 97.5906) (width 0.508) (layer B.Cu) (net 4))
+  (segment (start 108.332 79.6582) (end 108.332 81.5778) (width 0.508) (layer B.Cu) (net 4))
+  (segment (start 156.846 89.4254) (end 154.6498 91.6216) (width 0.508) (layer F.Cu) (net 4))
+  (segment (start 130.3138 91.6216) (end 124.3448 97.5906) (width 0.508) (layer F.Cu) (net 4))
+  (segment (start 154.6498 91.6216) (end 130.3138 91.6216) (width 0.508) (layer F.Cu) (net 4))
   (segment (start 132.982699 60.087499) (end 138.0754 65.1802) (width 0.254) (layer B.Cu) (net 9))
   (segment (start 132.982699 55.383927) (end 132.982699 60.087499) (width 0.254) (layer B.Cu) (net 9))
