File: Hardware/tool_circuit/tool_circuit.kicad_pcb (KiCad board)
At the start: 2 copper layers, 65.2 x 62.6 mm, 33 parts, among them J1 EJ503A, J2 Temp_Sense, J3 Accel., J4 GPIO_CONNECTOR, SW1 Switch, U1 LM2576D2TR4-5G

Commit message: Updated Gerbers
Other:
- board text added: "J4"

Commit message: pcb
Parts:
- removed CR1: B380-13-F, B380-13-F:B380-13-F
- removed R7: 100, footprints:RNCP1206FTD100R
- added CR2: B380-13-F, B380-13-F:B380-13-F, F.Cu at (116.8, 63.2)
- added R1: 10k, RNCP1206FTD10K0:RESC3115X60N, F.Cu at (132.5, 46.1)
- L1: value 100 uH -> 100uH
- R3: value 10k -> 100; footprint RNCP1206FTD10K0:RESC3115X60N -> RNCP1206FTD100R:RESC3115X60N
- R5, R6: footprint footprints:RNCP1206FTD100R -> RNCP1206FTD100R:RESC3115X60N
- TP1: value Vin_tp -> Vin
- TP2: value 5V_Reg_Vout_tp -> 5V_Reg_Vout
- TP3: value Tool_In_Use_tp -> Tool_In_Use
- TP4: value 3.3V_tp -> 3.3V
- TP5: value GPIO1_tp -> GPIO1
- TP6: value Disable_tp -> Disable
- TP7: value Enable_LED_tp -> Enable_LED
- TP8: value Data_Transfer_tp -> Data_Transfer
- moved R3 30.6 mm to (120.1, 87.3), turned to 0 degrees
- moved R5 12.7 mm to (133.1, 85.6)
- moved R6 9.89 mm to (143.4, 86.0)
- moved TP6 3.45 mm to (129.1, 73.2)
- moved LED1 2.32 mm to (151.9, 60.2)
- moved C2 0.86 mm to (106.5, 96.8)
- moved L1 0.51 mm to (130.6, 64.4)
Connections:
- J4 pad 15: GPIO22_GEN3 -> /raspberrypi_header.sch/GPIO22_GEN3
- LED1 pad 2: GPIO22_GEN3 -> Time_of_use
- R3 pad 1: Net-(R3-Pad1) -> Net-(D1-PadC)
- R5 pad 1: Net-(D1-PadC) -> Net-(D2-Pad1)
- R6 pad 1: Net-(D2-Pad1) -> Net-(D3-PadC)
- SW1 pad 1: +5V -> +3V3
- SW1 pad 2: GPIO22_GEN3 -> Time_of_use
- SW1 pad 3: Net-(R3-Pad1) -> GND
- TP3 pad 1: GPIO22_GEN3 -> Time_of_use
Routing:
- net GPIO22_GEN3: track 112.1 -> 0.00 mm
- net Time_of_use: track 0.00 -> 98.7 mm, vias 0 -> 1
- net +5V: track 155.7 -> 114.6 mm, vias 4 -> 3
- net GND: track 6.13 -> 32.5 mm
- net +3V3: track 116.8 -> 129.7 mm, vias 2 -> 3
- net /raspberrypi_header.sch/GPIO22_GEN3: track 0.00 -> 10.6 mm
- net Net-(R3-Pad1): track 8.49 -> 0.00 mm
- net /raspberrypi_header.sch/Disable_LED: track 41.9 -> 36.1 mm, vias 1 -> 3
- net Net-(D3-PadC): track 7.52 -> 5.89 mm
- net Net-(LED1-Pad1): track 6.97 -> 5.34 mm
- net Net-(D2-Pad1): track 7.09 -> 5.46 mm
- net Net-(CR2-Pad1): track 29.7 -> 31.1 mm
- net /raspberrypi_header.sch/Enable_LED: track 34.3 -> 33.3 mm, vias 3 -> 1

Commit message: pcb
Routing:
- net GND: vias 5 -> 8
Changed lines of the file:
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@@
     (thickness 1.6)
     (drawings 21)
-    (tracks 190)
+    (tracks 193)
     (zones 0)
     (modules 33)
@@
     (32 B.Adhes user hide)
     (33 F.Adhes user hide)
-    (34 B.Paste user hide)
-    (35 F.Paste user hide)
+    (34 B.Paste user)
+    (35 F.Paste user)
     (36 B.SilkS user hide)
     (37 F.SilkS user)
@@
     (visible_elements 7FFFFFFF)
     (pcbplotparams
-      (layerselection 0x010f0_ffffffff)
+      (layerselection 0x010fc_ffffffff)
       (usegerberextensions true)
       (usegerberattributes false)
@@
   (segment (start 112.104799 51.704601) (end 112.104799 53.604165) (width 0.254) (layer F.Cu) (net 1))
   (segment (start 113.3358 50.4736) (end 112.104799 51.704601) (width 0.254) (layer F.Cu) (net 1))
+  (via (at 121.9972 62.3862) (size 0.6858) (drill 0.3302) (layers F.Cu B.Cu) (net 1))
+  (via (at 122.9116 62.3862) (size 0.6858) (drill 0.3302) (layers F.Cu B.Cu) (net 1))
+  (via (at 121.0574 62.3862) (size 0.6858) (drill 0.3302) (layers F.Cu B.Cu) (net 1))
   (segment (start 126.874 85.424) (end 121.2098 79.7598) (width 0.508) (layer F.Cu) (net 2))
   (segment (start 126.874 88.0148) (end 126.874 85.424) (width 0.508) (layer F.Cu) (net 2))
