File: Hardware/tool_circuit/Accelerometer.sch (KiCad schematic (older format))
At the start: 1 part, among them J3 Accel.

Commit message: pcb
Changed lines of the file:
@@
 Text GLabel 6000 4000 0    50   BiDi ~ 0
 GPIO3_SCL1
+$Comp
+L power:PWR_FLAG #FLG0101
+U 1 1 61A519B5
+P 7050 3350
+F 0 "#FLG0101" H 7050 3425 50  0001 C CNN
+F 1 "PWR_FLAG" H 7050 3523 50  0000 C CNN
+F 2 "" H 7050 3350 50  0001 C CNN
+F 3 "~" H 7050 3350 50  0001 C CNN
+	1    7050 3350
+	1    0    0    -1
+$EndComp
+$Comp
+L power:GND #PWR0102
+U 1 1 61A5202B
+P 7050 3350
+F 0 "#PWR0102" H 7050 3100 50  0001 C CNN
+F 1 "GND" H 7055 3177 50  0000 C CNN
+F 2 "" H 7050 3350 50  0001 C CNN
+F 3 "" H 7050 3350 50  0001 C CNN
+	1    7050 3350
+	1    0    0    -1
+$EndComp
 $EndSCHEMATC
