File: Hardware/tool_circuit/_autosave-raspberrypi_header.sch (KiCad schematic (older format))
At the start: 20 parts, among them J4 GPIO_CONNECTOR

Commit message: pcb
Connections:
- net GPIO22_GEN3: no longer LED1.2, R1.1, TP3.1
- new net Time_of_use: LED1.2, R1.1, TP3.1
Changed lines of the file:
@@
 Wire Wire Line
 	7000 2000 7100 2000
-Text Label 3600 2750 0    50   ~ 0
-Tool_In_Use
 Text Label 4100 2250 0    50   ~ 0
 GPIO3_SCL1
@@
 GPIO27_GEN2
 Text GLabel 2050 2750 0    50   BiDi ~ 0
-GPIO22_GEN3
+Time_of_use
 Wire Wire Line
 	5050 2650 2750 2650
